Commit message: update to load successfully velocity controller

File: ur_description/urdf/common.gazebo.xacro (robot description, xacro)
@@ -2,8 +2,8 @@
 <robot xmlns:xacro="http://wiki.ros.org/xacro">
   <gazebo>
-      <plugin name="ros_control" filename="libhwi_switch_gazebo_ros_control.so">
-          <robotNamespace>""</robotNamespace>
-          <!--filterJointsParam>joint_names</filterJointsParam-->
-      </plugin>
+    <plugin name="ros_control" filename="libgazebo_ros_control.so">
+      <!--robotNamespace>/</robotNamespace-->
+      <!--robotSimType>gazebo_ros_control/DefaultRobotHWSim</robotSimType-->
+    </plugin>
 <!--
     <plugin name="gazebo_ros_power_monitor_controller" filename="libgazebo_ros_power_monitor.so">

File: ur_description/urdf/ur10VelControl.urdf.xacro (robot description, xacro)
@@ -7,4 +7,41 @@
   <xacro:include filename="$(find ur_description)/urdf/urVelControl.transmission.xacro" />
   <xacro:include filename="$(find ur_description)/urdf/urVelControl.gazebo.xacro" />
+  <xacro:property name="pi" value="3.14159265" />
+  <!-- Inertia parameters -->
+  <xacro:property name="base_mass" value="4.0" />  <!-- This mass might be incorrect -->
+  <xacro:property name="shoulder_mass" value="1" />
+  <xacro:property name="upper_arm_mass" value="1" />
+  <xacro:property name="forearm_mass" value="1" />
+  <xacro:property name="wrist_1_mass" value="0.5" />
+  <xacro:property name="wrist_2_mass" value="0.5" />
+  <xacro:property name="wrist_3_mass" value="0.5" />
+  <!-- These parameters are borrowed from the urcontrol.conf file
+       but are not verified for the correct permutation.
+       The permutation was guessed by looking at the UR5 parameters.
+       Serious use of these parameters needs further inspection. -->
+  <xacro:property name="shoulder_cog" value="0.00008 0.00244 -0.037" />
+  <xacro:property name="upper_arm_cog" value="0.00001 0.15061 0.38757" />
+  <xacro:property name="forearm_cog" value="-0.00012 0.06112 0.1984" />
+  <xacro:property name="wrist_1_cog" value="-0.00021 -0.00112 0.02269" />
+  <xacro:property name="wrist_2_cog" value="-0.00021 0.00112 0.002269" />
+  <xacro:property name="wrist_3_cog" value="0 -0.001156 -0.00149" />
+  <!-- Kinematic model -->
+  <!-- Properties from urcontrol.conf -->
+  <xacro:property name="ur10_d1" value="0.1273" />
+  <xacro:property name="ur10_a2" value="-0.612" />
+  <xacro:property name="ur10_a3" value="-0.5723" />
+  <xacro:property name="ur10_d4" value="0.163941" />
+  <xacro:property name="ur10_d5" value="0.1157" />
+  <xacro:property name="ur10_d6" value="0.0922" />
+  <!-- Arbitrary offsets for shoulder/elbow joints -->
+  <xacro:property name="shoulder_offset" value="0.220941" />  <!-- measured from model -->
+  <xacro:property name="elbow_offset" value="-0.1719" /> <!-- measured from model -->
+  <!-- link lengths used in model -->
+  <xacro:property name="shoulder_height" value="${ur10_d1}" />
+  <xacro:property name="upper_arm_length" value="${-ur10_a2}" />
+  <xacro:property name="forearm_length" value="${-ur10_a3}" />
+  <xacro:property name="wrist_1_length" value="${ur10_d4 - elbow_offset - shoulder_offset}" />
+  <xacro:property name="wrist_2_length" value="${ur10_d5}" />
+  <xacro:property name="wrist_3_length" value="${ur10_d6}" />
   <xacro:macro name="cylinder_inertial" params="radius length mass *origin">
     <inertial>
@@ -16,50 +53,11 @@
     </inertial>
   </xacro:macro>
-  <xacro:macro name="ur10VelControl_robot" params="prefix joint_limited
-    shoulder_pan_lower_limit:=${-pi}    shoulder_pan_upper_limit:=${pi}
-    shoulder_lift_lower_limit:=${-pi}    shoulder_lift_upper_limit:=${pi}
-    elbow_joint_lower_limit:=${-pi}    elbow_joint_upper_limit:=${pi}
-    wrist_1_lower_limit:=${-pi}    wrist_1_upper_limit:=${pi}
-    wrist_2_lower_limit:=${-pi}    wrist_2_upper_limit:=${pi}
-    wrist_3_lower_limit:=${-pi}    wrist_3_upper_limit:=${pi}
-    safety_limits:=false safety_pos_margin:=0.15
-    safety_k_position:=20">
-    <!-- Inertia parameters -->
-    <xacro:property name="base_mass" value="4.0" />  <!-- This mass might be incorrect -->
-    <xacro:property name="shoulder_mass" value="7.778" />
-    <xacro:property name="upper_arm_mass" value="12.93" />
-    <xacro:property name="forearm_mass" value="3.87" />
-    <xacro:property name="wrist_1_mass" value="1.96" />
-    <xacro:property name="wrist_2_mass" value="1.96" />
-    <xacro:property name="wrist_3_mass" value="0.202" />
-    <!-- These parameters are borrowed from the urcontrol.conf file
-        but are not verified for the correct permutation.
-        The permutation was guessed by looking at the UR5 parameters.
-        Serious use of these parameters needs further inspection. -->
-    <xacro:property name="shoulder_cog" value="0.00008 0.00244 -0.037" />
-    <xacro:property name="upper_arm_cog" value="0.00001 0.15061 0.38757" />
-    <xacro:property name="forearm_cog" value="-0.00012 0.06112 0.1984" />
-    <xacro:property name="wrist_1_cog" value="-0.00021 -0.00112 0.02269" />
-    <xacro:property name="wrist_2_cog" value="-0.00021 0.00112 0.002269" />
-    <xacro:property name="wrist_3_cog" value="0 -0.001156 -0.00149" />
-    <!-- Kinematic model -->
-    <!-- Properties from urcontrol.conf -->
-    <xacro:property name="d1" value="0.1273" />
-    <xacro:property name="a2" value="-0.612" />
-    <xacro:property name="a3" value="-0.5723" />
-    <xacro:property name="d4" value="0.163941" />
-    <xacro:property name="d5" value="0.1157" />
-    <xacro:property name="d6" value="0.0922" />
-    <!-- Arbitrary offsets for shoulder/elbow joints -->
-    <xacro:property name="shoulder_offset" value="0.220941" />  <!-- measured from model -->
-    <xacro:property name="elbow_offset" value="-0.1719" /> <!-- measured from model -->
-    <xacro:property name="upper_arm_inertia_offset" value="0.045" />  <!-- measured from model -->
-    <!-- link lengths used in model -->
-    <xacro:property name="shoulder_height" value="${d1}" />
-    <xacro:property name="upper_arm_length" value="${-a2}" />
-    <xacro:property name="forearm_length" value="${-a3}" />
-    <xacro:property name="wrist_1_length" value="${d4 - elbow_offset - shoulder_offset}" />
-    <xacro:property name="wrist_2_length" value="${d5}" />
-    <xacro:property name="wrist_3_length" value="${d6}" />
+  <xacro:macro name="ur10_robot" params="prefix joint_limited
+                 shoulder_pan_lower_limit:=${-0.5*pi}    shoulder_pan_upper_limit:=${0.2}
+                 shoulder_lift_lower_limit:=${-pi}    shoulder_lift_upper_limit:=${pi}
+                 elbow_joint_lower_limit:=${-pi}    elbow_joint_upper_limit:=${0.2}
+                 wrist_1_lower_limit:=${-2*pi}    wrist_1_upper_limit:=${-0.5}
+                 wrist_2_lower_limit:=${-pi}    wrist_2_upper_limit:=${pi}
+                 wrist_3_lower_limit:=${0.5-pi}    wrist_3_upper_limit:=${0.5*pi}">
     <link name="${prefix}base_link" >
       <visual>
@@ -80,6 +78,5 @@
       </xacro:cylinder_inertial>
     </link>
-    <!--joint name="${prefix}shoulder_pan_joint" type="revolute"-->
-    <joint name="${prefix}joint_1" type="revolute">
+    <joint name="${prefix}shoulder_pan_joint" type="revolute">
       <parent link="${prefix}base_link" />
       <child link = "${prefix}shoulder_link" />
@@ -87,14 +84,8 @@
       <axis xyz="0 0 1" />
       <xacro:unless value="${joint_limited}">
-        <limit lower="${-2.0 * pi}" upper="${2.0 * pi}" effort="330.0" velocity="2.16"/>
-        <xacro:if value="${safety_limits}">
-          <safety_controller soft_lower_limit="${-2.0 * pi + safety_pos_margin}" soft_upper_limit="${2.0 * pi - safety_pos_margin}" k_position="${safety_k_position}" k_velocity="0.0"/>
-        </xacro:if>
-      </xacro:unless>
-      <xacro:if value="${joint_limited}">
-        <limit lower="${shoulder_pan_lower_limit}" upper="${shoulder_pan_upper_limit}" effort="330.0" velocity="2.16"/>
-        <xacro:if value="${safety_limits}">
-          <safety_controller soft_lower_limit="${shoulder_pan_lower_limit + safety_pos_margin}" soft_upper_limit="${shoulder_pan_upper_limit - safety_pos_margin}" k_position="${safety_k_position}" k_velocity="0.0"/>
-        </xacro:if>
+        <limit lower="${-2.0 * pi}" upper="${2.0 * pi}" effort="330.0" velocity="2.0"/>
+      </xacro:unless>
+      <xacro:if value="${joint_limited}">
+        <limit lower="${shoulder_pan_lower_limit}" upper="${shoulder_pan_upper_limit}" effort="330.0" velocity="2.0"/>
       </xacro:if>
       <dynamics damping="0.0" friction="0.0"/>
@@ -118,6 +109,5 @@
       </xacro:cylinder_inertial>
     </link>
-    <!--joint name="${prefix}shoulder_lift_joint" type="revolute"-->
-    <joint name="${prefix}joint_2" type="revolute">
+    <joint name="${prefix}shoulder_lift_joint" type="revolute">
       <parent link="${prefix}shoulder_link" />
       <child link = "${prefix}upper_arm_link" />
@@ -125,14 +115,8 @@
       <axis xyz="0 1 0" />
       <xacro:unless value="${joint_limited}">
-        <limit lower="${-2.0 * pi}" upper="${2.0 * pi}" effort="330.0" velocity="2.16"/>
-        <xacro:if value="${safety_limits}">
-          <safety_controller soft_lower_limit="${-2.0 * pi + safety_pos_margin}" soft_upper_limit="${2.0 * pi - safety_pos_margin}" k_position="${safety_k_position}" k_velocity="0.0"/>
-        </xacro:if>
-      </xacro:unless>
-      <xacro:if value="${joint_limited}">
-        <limit lower="${shoulder_lift_lower_limit}" upper="${shoulder_lift_upper_limit}" effort="330.0" velocity="2.16"/>
-        <xacro:if value="${safety_limits}">
-          <safety_controller soft_lower_limit="${shoulder_lift_lower_limit + safety_pos_margin}" soft_upper_limit="${shoulder_lift_upper_limit - safety_pos_margin}" k_position="${safety_k_position}" k_velocity="0.0"/>
-        </xacro:if>
+        <limit lower="${-2.0 * pi}" upper="${2.0 * pi}" effort="330.0" velocity="2.0"/>
+      </xacro:unless>
+      <xacro:if value="${joint_limited}">
+        <limit lower="${shoulder_lift_lower_limit}" upper="${shoulder_lift_upper_limit}" effort="330.0" velocity="2.0"/>
       </xacro:if>
       <dynamics damping="0.0" friction="0.0"/>
@@ -152,10 +136,9 @@
         </geometry>
       </collision>
-      <xacro:cylinder_inertial radius="0.075" length="${-a2}" mass="${upper_arm_mass}">
-        <origin xyz="0.0 ${-upper_arm_inertia_offset} ${-a2/2.0}" rpy="0 0 0" />
-      </xacro:cylinder_inertial>
-    </link>
-    <!--joint name="${prefix}elbow_joint" type="revolute"-->
-    <joint name="${prefix}joint_3" type="revolute">
+      <xacro:cylinder_inertial radius="0.075" length="${-ur10_a2}" mass="${upper_arm_mass}">
+        <origin xyz="0.0 0.0 ${-ur10_a2/2.0}" rpy="0 0 0" />
+      </xacro:cylinder_inertial>
+    </link>
+    <joint name="${prefix}elbow_joint" type="revolute">
       <parent link="${prefix}upper_arm_link" />
       <child link = "${prefix}forearm_link" />
@@ -163,14 +146,8 @@
       <axis xyz="0 1 0" />
       <xacro:unless value="${joint_limited}">
-        <limit lower="${-pi}" upper="${pi}" effort="150.0" velocity="3.15"/>
-        <xacro:if value="${safety_limits}">
-          <safety_controller soft_lower_limit="${-2.0 * pi + safety_pos_margin}" soft_upper_limit="${2.0 * pi - safety_pos_margin}" k_position="${safety_k_position}" k_velocity="0.0"/>
-        </xacro:if>
-      </xacro:unless>
-      <xacro:if value="${joint_limited}">
-        <limit lower="${elbow_joint_lower_limit}" upper="${elbow_joint_upper_limit}" effort="150.0" velocity="3.15"/>
-        <xacro:if value="${safety_limits}">
-          <safety_controller soft_lower_limit="${elbow_joint_lower_limit + safety_pos_margin}" soft_upper_limit="${elbow_joint_upper_limit - safety_pos_margin}" k_position="${safety_k_position}" k_velocity="0.0"/>
-        </xacro:if>
+        <limit lower="${-2.0 * pi}" upper="${2.0 * pi}" effort="150.0" velocity="2.0"/>
+      </xacro:unless>
+      <xacro:if value="${joint_limited}">
+        <limit lower="${elbow_joint_lower_limit}" upper="${elbow_joint_upper_limit}" effort="150.0" velocity="2.0"/>
       </xacro:if>
       <dynamics damping="0.0" friction="0.0"/>
@@ -190,10 +167,9 @@
         </geometry>
       </collision>
-      <xacro:cylinder_inertial radius="0.075" length="${-a3}" mass="${forearm_mass}">
-        <origin xyz="0.0 0.0 ${-a3/2.0}" rpy="0 0 0" />
-      </xacro:cylinder_inertial>
-    </link>
-    <!--joint name="${prefix}wrist_1_joint" type="revolute"-->
-    <joint name="${prefix}joint_4" type="revolute">
+      <xacro:cylinder_inertial radius="0.075" length="${-ur10_a3}" mass="${forearm_mass}">
+        <origin xyz="0.0 0.0 ${-ur10_a3/2.0}" rpy="0 0 0" />
+      </xacro:cylinder_inertial>
+    </link>
+    <joint name="${prefix}wrist_1_joint" type="revolute">
       <parent link="${prefix}forearm_link" />
       <child link = "${prefix}wrist_1_link" />
@@ -201,14 +177,8 @@
       <axis xyz="0 1 0" />
       <xacro:unless value="${joint_limited}">
-        <limit lower="${-2.0 * pi}" upper="${2.0 * pi}" effort="54.0" velocity="3.2"/>
-        <xacro:if value="${safety_limits}">
-          <safety_controller soft_lower_limit="${-2.0 * pi + safety_pos_margin}" soft_upper_limit="${2.0 * pi - safety_pos_margin}" k_position="${safety_k_position}" k_velocity="0.0"/>
-        </xacro:if>
-      </xacro:unless>
-      <xacro:if value="${joint_limited}">
-        <limit lower="${wrist_1_lower_limit}" upper="${wrist_1_upper_limit}" effort="54.0" velocity="3.2"/>
-        <xacro:if value="${safety_limits}">
-          <safety_controller soft_lower_limit="${wrist_1_lower_limit + safety_pos_margin}" soft_upper_limit="${wrist_1_upper_limit - safety_pos_margin}" k_position="${safety_k_position}" k_velocity="0.0"/>
-        </xacro:if>
+        <limit lower="${-2.0 * pi}" upper="${2.0 * pi}" effort="54.0" velocity="2.0"/>
+      </xacro:unless>
+      <xacro:if value="${joint_limited}">
+        <limit lower="${wrist_1_lower_limit}" upper="${wrist_1_upper_limit}" effort="54.0" velocity="2.0"/>
       </xacro:if>
       <dynamics damping="0.0" friction="0.0"/>
@@ -229,9 +199,8 @@
       </collision>
       <xacro:cylinder_inertial radius="0.075" length="0.12" mass="${wrist_1_mass}">
-        <origin xyz="0.0 ${wrist_1_length} 0.0" rpy="0 0 0" />
-      </xacro:cylinder_inertial>
-    </link>
-    <!--joint name="${prefix}wrist_2_joint" type="revolute"-->
-    <joint name="${prefix}joint_5" type="revolute">
+        <origin xyz="0.0 0.0 0.0" rpy="0 0 0" />
+      </xacro:cylinder_inertial>
+    </link>
+    <joint name="${prefix}wrist_2_joint" type="revolute">
       <parent link="${prefix}wrist_1_link" />
       <child link = "${prefix}wrist_2_link" />
@@ -239,14 +208,8 @@
       <axis xyz="0 0 1" />
       <xacro:unless value="${joint_limited}">
-        <limit lower="${-2.0 * pi}" upper="${2.0 * pi}" effort="54.0" velocity="3.2"/>
-        <xacro:if value="${safety_limits}">
-          <safety_controller soft_lower_limit="${-2.0 * pi + safety_pos_margin}" soft_upper_limit="${2.0 * pi - safety_pos_margin}" k_position="${safety_k_position}" k_velocity="0.0"/>
-        </xacro:if>
-      </xacro:unless>
-      <xacro:if value="${joint_limited}">
-        <limit lower="${wrist_2_lower_limit}" upper="${wrist_2_upper_limit}" effort="54.0" velocity="3.2"/>
-        <xacro:if value="${safety_limits}">
-          <safety_controller soft_lower_limit="${wrist_2_lower_limit + safety_pos_margin}" soft_upper_limit="${wrist_2_upper_limit - safety_pos_margin}" k_position="${safety_k_position}" k_velocity="0.0"/>
-        </xacro:if>
+        <limit lower="${-2.0 * pi}" upper="${2.0 * pi}" effort="54.0" velocity="2.0"/>
+      </xacro:unless>
+      <xacro:if value="${joint_limited}">
+        <limit lower="${wrist_2_lower_limit}" upper="${wrist_2_upper_limit}" effort="54.0" velocity="2.0"/>
       </xacro:if>
       <dynamics damping="0.0" friction="0.0"/>
@@ -267,9 +230,8 @@
       </collision>
       <xacro:cylinder_inertial radius="0.075" length="0.12" mass="${wrist_2_mass}">
-        <origin xyz="0.0 0.0 ${wrist_2_length}" rpy="0 0 0" />
-      </xacro:cylinder_inertial>
-    </link>
-    <!--joint name="${prefix}wrist_3_joint" type="revolute"-->
-    <joint name="${prefix}joint_6" type="revolute">
+        <origin xyz="0.0 0.0 0.0" rpy="0 0 0" />
+      </xacro:cylinder_inertial>
+    </link>
+    <joint name="${prefix}wrist_3_joint" type="revolute">
       <parent link="${prefix}wrist_2_link" />
       <child link = "${prefix}wrist_3_link" />
@@ -277,14 +239,8 @@
       <axis xyz="0 1 0" />
       <xacro:unless value="${joint_limited}">
-        <limit lower="${-2.0 * pi}" upper="${2.0 * pi}" effort="54.0" velocity="3.2"/>
-        <xacro:if value="${safety_limits}">
-          <safety_controller soft_lower_limit="${-2.0 * pi + safety_pos_margin}" soft_upper_limit="${2.0 * pi - safety_pos_margin}" k_position="${safety_k_position}" k_velocity="0.0"/>
-        </xacro:if>
-      </xacro:unless>
-      <xacro:if value="${joint_limited}">
-        <limit lower="${wrist_3_lower_limit}" upper="${wrist_3_upper_limit}" effort="54.0" velocity="3.2"/>
-        <xacro:if value="${safety_limits}">
-          <safety_controller soft_lower_limit="${wrist_3_lower_limit + safety_pos_margin}" soft_upper_limit="${wrist_3_upper_limit - safety_pos_margin}" k_position="${safety_k_position}" k_velocity="0.0"/>
-        </xacro:if>
+        <limit lower="${-2.0 * pi}" upper="${2.0 * pi}" effort="54.0" velocity="2.0"/>
+      </xacro:unless>
+      <xacro:if value="${joint_limited}">
+        <limit lower="${wrist_3_lower_limit}" upper="${wrist_3_upper_limit}" effort="54.0" velocity="2.0"/>
       </xacro:if>
       <dynamics damping="0.0" friction="0.0"/>
@@ -304,6 +260,6 @@
         </geometry>
       </collision>
-      <xacro:cylinder_inertial radius="0.045" length="0.0305" mass="${wrist_3_mass}">
-        <origin xyz="0.0 ${wrist_3_length - 0.0305/2} 0.0" rpy="${pi/2} 0 0" />
+      <xacro:cylinder_inertial radius="0.075" length="0.12" mass="${wrist_3_mass}">
+        <origin xyz="0.0 0.0 0.0" rpy="0 0 0" />
       </xacro:cylinder_inertial>
     </link>
@@ -321,6 +277,6 @@
       </collision>
     </link>
-    <xacro:urVelControl_arm_transmission prefix="${prefix}"/>
-    <xacro:urVelControl_arm_gazebo prefix="${prefix}" />
+    <xacro:ur_arm_transmission prefix="${prefix}" />
+    <xacro:ur_arm_gazebo prefix="${prefix}" />
     <!-- ROS base_link to UR 'Base' Coordinates transform -->
     <link name="${prefix}base"/>
@@ -335,17 +291,24 @@
     </joint>
     <!-- Frame coincident with all-zeros TCP on UR controller -->
-    <link name="${prefix}tool0"/>
+    <link name="${prefix}tool0">
+      <collision>
+        <geometry>
+          <box size="0.01 0.01 0.01"/>
+        </geometry>
+        <origin rpy="0 0 0" xyz="-0.01 0 0"/>
+      </collision>
+    </link>
     <joint name="${prefix}wrist_3_link-tool0_fixed_joint" type="fixed">
-      <origin xyz="0 ${wrist_3_length} 0" rpy="${pi/-2.0} 0 0"/>
+      <origin xyz="0.0 ${wrist_3_length+0.14} 0.0" rpy="0.0 0.0 ${pi/2.0}" />
       <parent link="${prefix}wrist_3_link"/>
       <child link="${prefix}tool0"/>
-    </joint>
-    <!-- ros_control plugin -->
-    <gazebo>
-      <plugin name="ros_control" filename="libhwi_switch_gazebo_ros_control.so">
-          <robotNamespace>"${prefix}"</robotNamespace>
-          <filterJointsParam>joint_names</filterJointsParam>
-      </plugin>
-    </gazebo>
+      <xacro:unless value="${joint_limited}">
+        <limit lower="${-2.0 * pi}" upper="${2.0 * pi}" effort="54.0" velocity="3.2"/>
+      </xacro:unless>
+      <xacro:if value="${joint_limited}">
+        <limit lower="${wrist_3_lower_limit}" upper="${wrist_3_upper_limit}" effort="54.0" velocity="3.2"/>
+      </xacro:if>
+      <dynamics damping="0.0" friction="0.0"/>
+    </joint>
   </xacro:macro>
 </robot>

File: ur_description/urdf/ur10VelControl_robot.urdf.xacro (robot description, xacro)
@@ -1,11 +1,16 @@
 <?xml version="1.0"?>
-<robot xmlns:xacro="http://wiki.ros.org/xacro" name="ur10" >
+<robot xmlns:xacro="http://ros.org/wiki/xacro"
+       name="ur10" >
   <!-- common stuff -->
-  <!--xacro:include filename="$(find ur_description)/urdf/common.gazebo.xacro" /-->
+  <xacro:include filename="$(find ur_description)/urdf/common.gazebo.xacro" />
   <!-- ur10 -->
   <xacro:include filename="$(find ur_description)/urdf/ur10VelControl.urdf.xacro" />
-  <!-- arm -->
-  <xacro:ur10VelControl_robot prefix="" joint_limited="false"/>
-  <link name="world" />
+  <!--link name="world" />
+  <joint name="world_joint" type="fixed">
+    <parent link="world" />
+    <child link = "arm_base_link" />
+    <origin xyz="0.0 0.0 0.0" rpy="0.0 0.0 0.0" />
+  </joint-->
+ <link name="world" />
   <joint name="world-robot_base_joint" type="fixed">
     <origin xyz="-0.50 -0.30 0.30" rpy="0 0 0" />
@@ -26,6 +31,15 @@
   <joint name="world_joint" type="fixed">
     <parent link="robot_base" />
-    <child link = "base_link" />
+    <child link = "arm_base_link" />
     <origin xyz="0.324 -0.191 0.2925" rpy="0.0 0.0 -2.3562" />
   </joint>
+  <!-- arm -->
+  <xacro:ur10_robot prefix="arm_" joint_limited="false"/>
+  <!-- ros_control plugin -->
+  <gazebo>
+    <plugin name="ros_control" filename="libhwi_switch_gazebo_ros_control.so">
+      <robotNamespace>arm</robotNamespace>
+      <filterJointsParam>joint_names</filterJointsParam>
+    </plugin>
+  </gazebo>
 </robot>

File: ur_description/urdf/urVelControl.gazebo.xacro (robot description, xacro)
@@ -1,26 +1,20 @@
 <?xml version="1.0"?>
-<robot xmlns:xacro="http://wiki.ros.org/xacro">
-  <xacro:macro name="urVelControl_arm_gazebo" params="prefix">
-    <gazebo reference="${prefix}shoulder_link">
-      <selfCollide>true</selfCollide>
-    </gazebo>
-    <gazebo reference="${prefix}upper_arm_link">
-      <selfCollide>true</selfCollide>
-    </gazebo>
-    <gazebo reference="${prefix}forearm_link">
-      <selfCollide>true</selfCollide>
-    </gazebo>
-    <gazebo reference="${prefix}wrist_1_link">
-      <selfCollide>true</selfCollide>
-    </gazebo>
-    <gazebo reference="${prefix}wrist_3_link">
-      <selfCollide>true</selfCollide>
-    </gazebo>
-    <gazebo reference="${prefix}wrist_2_link">
-      <selfCollide>true</selfCollide>
-    </gazebo>
-    <gazebo reference="${prefix}ee_link">
-      <selfCollide>true</selfCollide>
-    </gazebo>
+<robot xmlns:xacro="http://ros.org/wiki/xacro">
+  <xacro:macro name="ur_arm_gazebo" params="prefix">
+    <!--gazebo reference="${prefix}ee_link">
+      <self_collide>false</self_collide>
+      <sensor name='${prefix}ee_link_sensor' type='contact'>
+        <always_on>true</always_on>
+        <update_rate>100.0</update_rate>
+        <contact>
+          <collision>${prefix}ee_link_collision</collision>
+          <topic>${prefix}ee_link_bumper</topic>
+        </contact>
+        <plugin name="${prefix}ee_link_gazebo_ros_bumper_controller" filename="libgazebo_ros_bumper.so">
+          <bodyName>${prefix}ee_link</bodyName>
+          <bumperTopicName>${prefix}ee_link_bumper</bumperTopicName>
+        </plugin>
+      </sensor>
+    </gazebo-->
   </xacro:macro>
 </robot>
