Commit message: renaming of the shoulder joint names

File: ur_description/urdf/ur.transmission.xacro (robot description, xacro)
@@ -2,28 +2,28 @@
 <robot xmlns:xacro="http://ros.org/wiki/xacro">
   <xacro:macro name="ur_arm_transmission" params="prefix">
-    <transmission name="${prefix}shoulder_pan_trans">
+    <transmission name="${prefix}shoulder_1_trans">
       <type>transmission_interface/SimpleTransmission</type>
-      <joint name="${prefix}shoulder_pan_joint">
+      <joint name="${prefix}shoulder_1_joint">
         <hardwareInterface>PositionJointInterface</hardwareInterface>
       </joint>
-      <actuator name="${prefix}shoulder_pan_motor">
+      <actuator name="${prefix}shoulder_1_motor">
         <mechanicalReduction>1</mechanicalReduction>
       </actuator>
     </transmission>
-    <transmission name="${prefix}shoulder_lift_trans">
+    <transmission name="${prefix}shoulder_2_trans">
       <type>transmission_interface/SimpleTransmission</type>
-      <joint name="${prefix}shoulder_lift_joint">
+      <joint name="${prefix}shoulder_2_joint">
         <hardwareInterface>PositionJointInterface</hardwareInterface>
       </joint>
-      <actuator name="${prefix}shoulder_lift_motor">
+      <actuator name="${prefix}shoulder_2_motor">
         <mechanicalReduction>1</mechanicalReduction>
       </actuator>
     </transmission>
-    <transmission name="${prefix}elbow_trans">
+    <transmission name="${prefix}3_trans">
       <type>transmission_interface/SimpleTransmission</type>
-      <joint name="${prefix}elbow_joint">
+      <joint name="${prefix}3_joint">
         <hardwareInterface>PositionJointInterface</hardwareInterface>
       </joint>
-      <actuator name="${prefix}elbow_motor">
+      <actuator name="${prefix}3_motor">
         <mechanicalReduction>1</mechanicalReduction>
       </actuator>

File: ur_description/urdf/ur10.urdf.xacro (robot description, xacro)
@@ -54,6 +54,6 @@
   </xacro:macro>
   <xacro:macro name="ur10_robot" params="prefix joint_limited
-		 shoulder_pan_lower_limit:=${-0.5*pi}    shoulder_pan_upper_limit:=${0.5}
-		 shoulder_lift_lower_limit:=${-pi}    shoulder_lift_upper_limit:=${pi}
+		 shoulder_1_joint_lower_limit:=${-0.5*pi}    shoulder_1_joint_upper_limit:=${0.5}
+		 shoulder_2_joint_lower_limit:=${-pi}    shoulder_2_joint_upper_limit:=${pi}
 		 shoulder_3_joint_lower_limit:=${-pi}    shoulder_3_joint_upper_limit:=${0.2}
 		 wrist_1_lower_limit:=${-2*pi}    wrist_1_upper_limit:=${-0.5}
@@ -87,5 +87,5 @@
       </xacro:unless>
       <xacro:if value="${joint_limited}">
-        <limit lower="${shoulder_pan_lower_limit}" upper="${shoulder_pan_upper_limit}" effort="330.0" velocity="2.16"/>
+        <limit lower="${shoulder_1_joint_lower_limit}" upper="${shoulder_1_joint_upper_limit}" effort="330.0" velocity="2.16"/>
       </xacro:if>
       <dynamics damping="0.0" friction="0.0"/>
@@ -118,5 +118,5 @@
       </xacro:unless>
       <xacro:if value="${joint_limited}">
-        <limit lower="${shoulder_lift_lower_limit}" upper="${shoulder_lift_upper_limit}" effort="330.0" velocity="2.16"/>
+        <limit lower="${shoulder_2_joint_lower_limit}" upper="${shoulder_2_joint_upper_limit}" effort="330.0" velocity="2.16"/>
       </xacro:if>
       <dynamics damping="0.0" friction="0.0"/>

File: ur_description/urdf/ur10_joint_limited_robot.urdf.xacro (robot description, xacro)
@@ -8,6 +8,6 @@
   <!-- arm -->
   <xacro:ur10_robot prefix="" joint_limited="true"
-		 shoulder_1_lower_limit="${-pi}" shoulder_1_upper_limit="${pi}"
-		 shoulder_2_lower_limit="${-pi}" shoulder_2_upper_limit="${pi}"
+		 shoulder_1_joint_lower_limit="${-pi}" shoulder_1_joint_upper_limit="${pi}"
+		 shoulder_2_joint_lower_limit="${-pi}" shoulder_2_joint_upper_limit="${pi}"
 		 shoulder_3_joint_lower_limit="${-pi}" shoulder_3_joint_upper_limit="${pi}"
 		 wrist_1_lower_limit="${-pi}" wrist_1_upper_limit="${pi}"

Commit message: added hardwareInterface and attach bumper sensor

File: ur_description/urdf/ur.transmission.xacro (robot description, xacro)
@@ -6,4 +6,5 @@
       <joint name="${prefix}shoulder_pan_joint">
         <hardwareInterface>PositionJointInterface</hardwareInterface>
+        <hardwareInterface>VelocityJointInterface</hardwareInterface>
       </joint>
       <actuator name="${prefix}shoulder_pan_motor">
@@ -15,4 +16,5 @@
       <joint name="${prefix}shoulder_lift_joint">
         <hardwareInterface>PositionJointInterface</hardwareInterface>
+        <hardwareInterface>VelocityJointInterface</hardwareInterface>
       </joint>
       <actuator name="${prefix}shoulder_lift_motor">
@@ -24,4 +26,5 @@
       <joint name="${prefix}elbow_joint">
         <hardwareInterface>PositionJointInterface</hardwareInterface>
+        <hardwareInterface>VelocityJointInterface</hardwareInterface>
       </joint>
       <actuator name="${prefix}elbow_motor">
@@ -33,4 +36,5 @@
       <joint name="${prefix}wrist_1_joint">
         <hardwareInterface>PositionJointInterface</hardwareInterface>
+        <hardwareInterface>VelocityJointInterface</hardwareInterface>
       </joint>
       <actuator name="${prefix}wrist_1_motor">
@@ -42,4 +46,5 @@
       <joint name="${prefix}wrist_2_joint">
         <hardwareInterface>PositionJointInterface</hardwareInterface>
+        <hardwareInterface>VelocityJointInterface</hardwareInterface>
       </joint>
       <actuator name="${prefix}wrist_2_motor">
@@ -51,4 +56,5 @@
       <joint name="${prefix}wrist_3_joint">
         <hardwareInterface>PositionJointInterface</hardwareInterface>
+        <hardwareInterface>VelocityJointInterface</hardwareInterface>
       </joint>
       <actuator name="${prefix}wrist_3_motor">
@@ -56,4 +62,14 @@
       </actuator>
     </transmission>
+    <transmission name="${prefix}ee_fixed_trans">
+      <type>transmission_interface/SimpleTransmission</type>
+      <joint name="${prefix}ee_fixed_joint">
+        <hardwareInterface>PositionJointInterface</hardwareInterface>
+        <hardwareInterface>VelocityJointInterface</hardwareInterface>
+      </joint>
+      <actuator name="${prefix}ee_fixed_motor">
+        <mechanicalReduction>1</mechanicalReduction>
+      </actuator>
+    </transmission>
   </xacro:macro>
 </robot>

Commit message: rename joint name as original name

File: ur_description/urdf/ur.transmission.xacro (robot description, xacro)
@@ -2,28 +2,28 @@
 <robot xmlns:xacro="http://ros.org/wiki/xacro">
   <xacro:macro name="ur_arm_transmission" params="prefix">
-    <transmission name="${prefix}shoulder_1_trans">
+    <transmission name="${prefix}shoulder_pan_trans">
       <type>transmission_interface/SimpleTransmission</type>
-      <joint name="${prefix}shoulder_1_joint">
+      <joint name="${prefix}shoulder_pan_joint">
         <hardwareInterface>PositionJointInterface</hardwareInterface>
       </joint>
-      <actuator name="${prefix}shoulder_1_motor">
+      <actuator name="${prefix}shoulder_pan_motor">
         <mechanicalReduction>1</mechanicalReduction>
       </actuator>
     </transmission>
-    <transmission name="${prefix}shoulder_2_trans">
+    <transmission name="${prefix}shoulder_lift_trans">
       <type>transmission_interface/SimpleTransmission</type>
-      <joint name="${prefix}shoulder_2_joint">
+      <joint name="${prefix}shoulder_lift_joint">
         <hardwareInterface>PositionJointInterface</hardwareInterface>
       </joint>
-      <actuator name="${prefix}shoulder_2_motor">
+      <actuator name="${prefix}shoulder_lift_motor">
         <mechanicalReduction>1</mechanicalReduction>
       </actuator>
     </transmission>
-    <transmission name="${prefix}3_trans">
+    <transmission name="${prefix}elbow_trans">
       <type>transmission_interface/SimpleTransmission</type>
-      <joint name="${prefix}3_joint">
+      <joint name="${prefix}elbow_joint">
         <hardwareInterface>PositionJointInterface</hardwareInterface>
       </joint>
-      <actuator name="${prefix}3_motor">
+      <actuator name="${prefix}elbow_motor">
         <mechanicalReduction>1</mechanicalReduction>
       </actuator>

File: ur_description/urdf/ur10.urdf.xacro (robot description, xacro)
@@ -54,5 +54,5 @@
   </xacro:macro>
   <xacro:macro name="ur10_robot" params="prefix joint_limited
-		 shoulder_1_joint_lower_limit:=${-0.5*pi}    shoulder_1_joint_upper_limit:=${0.5}
+		 shoulder_1_joint_lower_limit:=${-pi}    shoulder_1_joint_upper_limit:=${0.5}
 		 shoulder_2_joint_lower_limit:=${-pi}    shoulder_2_joint_upper_limit:=${pi}
 		 shoulder_3_joint_lower_limit:=${-pi}    shoulder_3_joint_upper_limit:=${0.2}

File: ur_description/urdf/ur10_joint_limited_robot.urdf.xacro (robot description, xacro)
@@ -8,7 +8,7 @@
   <!-- arm -->
   <xacro:ur10_robot prefix="" joint_limited="true"
-		 shoulder_1_joint_lower_limit="${-pi}" shoulder_1_joint_upper_limit="${pi}"
-		 shoulder_2_joint_lower_limit="${-pi}" shoulder_2_joint_upper_limit="${pi}"
-		 shoulder_3_joint_lower_limit="${-pi}" shoulder_3_joint_upper_limit="${pi}"
+		 shoulder_pan_lower_limit="${-pi}" shoulder_pan_upper_limit="${pi}"
+		 shoulder_lift_lower_limit="${-pi}" shoulder_lift_upper_limit="${pi}"
+		 elbow_joint_lower_limit="${-pi}" elbow_joint_upper_limit="${pi}"
 		 wrist_1_lower_limit="${-pi}" wrist_1_upper_limit="${pi}"
 		 wrist_2_lower_limit="${-pi}" wrist_2_upper_limit="${pi}"

Commit message: rename_joint_names because modern driver set joint state accord to alphabatic order

File: ur_description/urdf/ur.transmission.xacro (robot description, xacro)
@@ -2,28 +2,28 @@
 <robot xmlns:xacro="http://ros.org/wiki/xacro">
   <xacro:macro name="ur_arm_transmission" params="prefix">
-    <transmission name="${prefix}shoulder_pan_trans">
+    <transmission name="${prefix}shoulder_1_trans">
       <type>transmission_interface/SimpleTransmission</type>
-      <joint name="${prefix}shoulder_pan_joint">
+      <joint name="${prefix}shoulder_1_joint">
         <hardwareInterface>PositionJointInterface</hardwareInterface>
       </joint>
-      <actuator name="${prefix}shoulder_pan_motor">
+      <actuator name="${prefix}shoulder_1_motor">
         <mechanicalReduction>1</mechanicalReduction>
       </actuator>
     </transmission>
-    <transmission name="${prefix}shoulder_lift_trans">
+    <transmission name="${prefix}shoulder_2_trans">
       <type>transmission_interface/SimpleTransmission</type>
-      <joint name="${prefix}shoulder_lift_joint">
+      <joint name="${prefix}shoulder_2_joint">
         <hardwareInterface>PositionJointInterface</hardwareInterface>
       </joint>
-      <actuator name="${prefix}shoulder_lift_motor">
+      <actuator name="${prefix}shoulder_2_motor">
         <mechanicalReduction>1</mechanicalReduction>
       </actuator>
     </transmission>
-    <transmission name="${prefix}elbow_trans">
+    <transmission name="${prefix}shoulder_3_trans">
       <type>transmission_interface/SimpleTransmission</type>
-      <joint name="${prefix}elbow_joint">
+      <joint name="${prefix}shoulder_3_joint">
         <hardwareInterface>PositionJointInterface</hardwareInterface>
       </joint>
-      <actuator name="${prefix}elbow_motor">
+      <actuator name="${prefix}shoulder_3_motor">
         <mechanicalReduction>1</mechanicalReduction>
       </actuator>

File: ur_description/urdf/ur10.urdf.xacro (robot description, xacro)
@@ -54,7 +54,7 @@
   </xacro:macro>
   <xacro:macro name="ur10_robot" params="prefix joint_limited
-		 shoulder_pan_lower_limit:=${-pi}    shoulder_pan_upper_limit:=${0.5}
-		 shoulder_lift_lower_limit:=${-pi}    shoulder_lift_upper_limit:=${pi}
-		 elbow_joint_lower_limit:=${-pi}    elbow_joint_upper_limit:=${0.2}
+		 shoulder_1_joint_lower_limit:=${-pi}    shoulder_1_joint_upper_limit:=${0.5}
+		 shoulder_2_joint_lower_limit:=${-pi}    shoulder_2_joint_upper_limit:=${pi}
+		 shoulder_3_joint_lower_limit:=${-pi}    shoulder_3_joint_upper_limit:=${0.2}
 		 wrist_1_lower_limit:=${-2*pi}    wrist_1_upper_limit:=${-0.5}
 		 wrist_2_lower_limit:=${-pi}    wrist_2_upper_limit:=${pi}
@@ -78,5 +78,5 @@
       </xacro:cylinder_inertial>
     </link>
-    <joint name="${prefix}shoulder_pan_joint" type="revolute">
+    <joint name="${prefix}shoulder_1_joint" type="revolute">
       <parent link="${prefix}base_link" />
       <child link = "${prefix}shoulder_link" />
@@ -87,5 +87,5 @@
       </xacro:unless>
       <xacro:if value="${joint_limited}">
-        <limit lower="${shoulder_pan_lower_limit}" upper="${shoulder_pan_upper_limit}" effort="330.0" velocity="2.0"/>
+        <limit lower="${shoulder_1_joint_lower_limit}" upper="${shoulder_1_joint_upper_limit}" effort="330.0" velocity="2.0"/>
       </xacro:if>
       <dynamics damping="0.0" friction="0.0"/>
@@ -109,5 +109,5 @@
       </xacro:cylinder_inertial>
     </link>
-    <joint name="${prefix}shoulder_lift_joint" type="revolute">
+    <joint name="${prefix}shoulder_2_joint" type="revolute">
       <parent link="${prefix}shoulder_link" />
       <child link = "${prefix}upper_arm_link" />
@@ -118,5 +118,5 @@
       </xacro:unless>
       <xacro:if value="${joint_limited}">
-        <limit lower="${shoulder_lift_lower_limit}" upper="${shoulder_lift_upper_limit}" effort="330.0" velocity="2.0"/>
+        <limit lower="${shoulder_2_joint_lower_limit}" upper="${shoulder_2_joint_upper_limit}" effort="330.0" velocity="2.0"/>
       </xacro:if>
       <dynamics damping="0.0" friction="0.0"/>
@@ -140,5 +140,5 @@
       </xacro:cylinder_inertial>
     </link>
-    <joint name="${prefix}elbow_joint" type="revolute">
+    <joint name="${prefix}shoulder_3_joint" type="revolute">
       <parent link="${prefix}upper_arm_link" />
       <child link = "${prefix}forearm_link" />
@@ -149,5 +149,5 @@
       </xacro:unless>
       <xacro:if value="${joint_limited}">
-        <limit lower="${elbow_joint_lower_limit}" upper="${elbow_joint_upper_limit}" effort="150.0" velocity="2.0"/>
+        <limit lower="${shoulder_3_joint_lower_limit}" upper="${shoulder_3_joint_upper_limit}" effort="150.0" velocity="2.0"/>
       </xacro:if>
       <dynamics damping="0.0" friction="0.0"/>

File: ur_description/urdf/ur10_joint_limited_robot.urdf.xacro (robot description, xacro)
@@ -8,7 +8,7 @@
   <!-- arm -->
   <xacro:ur10_robot prefix="" joint_limited="true"
-		 shoulder_pan_lower_limit="${-pi}" shoulder_pan_upper_limit="${pi}"
-		 shoulder_lift_lower_limit="${-pi}" shoulder_lift_upper_limit="${pi}"
-		 elbow_joint_lower_limit="${-pi}" elbow_joint_upper_limit="${pi}"
+		 shoulder_1_joint_lower_limit="${-pi}" shoulder_1_joint_upper_limit="${pi}"
+		 shoulder_2_joint_lower_limit="${-pi}" shoulder_2_joint_upper_limit="${pi}"
+		 shoulder_3_joint_lower_limit="${-pi}" shoulder_3_joint_upper_limit="${pi}"
 		 wrist_1_lower_limit="${-pi}" wrist_1_upper_limit="${pi}"
 		 wrist_2_lower_limit="${-pi}" wrist_2_upper_limit="${pi}"

Commit message: chnage joint name, to reduce effort for reordring

File: ur_description/urdf/ur.transmission.xacro (robot description, xacro)
@@ -2,55 +2,55 @@
 <robot xmlns:xacro="http://wiki.ros.org/xacro">
   <xacro:macro name="ur_arm_transmission" params="prefix hw_interface">
-    <transmission name="${prefix}shoulder_pan_trans">
+    <transmission name="${prefix}joint_1_trans">
       <type>transmission_interface/SimpleTransmission</type>
-      <joint name="${prefix}shoulder_pan_joint">
+      <joint name="${prefix}joint_1">
         <hardwareInterface>${hw_interface}</hardwareInterface>
       </joint>
-      <actuator name="${prefix}shoulder_pan_motor">
+      <actuator name="${prefix}joint_1_motor">
         <mechanicalReduction>1</mechanicalReduction>
       </actuator>
     </transmission>
-    <transmission name="${prefix}shoulder_lift_trans">
+    <transmission name="${prefix}joint_2_trans">
       <type>transmission_interface/SimpleTransmission</type>
-      <joint name="${prefix}shoulder_lift_joint">
+      <joint name="${prefix}joint_2">
         <hardwareInterface>${hw_interface}</hardwareInterface>
       </joint>
-      <actuator name="${prefix}shoulder_lift_motor">
+      <actuator name="${prefix}joint_2_motor">
         <mechanicalReduction>1</mechanicalReduction>
       </actuator>
     </transmission>
-    <transmission name="${prefix}elbow_trans">
+    <transmission name="${prefix}joint_3_trans">
       <type>transmission_interface/SimpleTransmission</type>
-      <joint name="${prefix}elbow_joint">
+      <joint name="${prefix}joint_3">
         <hardwareInterface>${hw_interface}</hardwareInterface>
       </joint>
-      <actuator name="${prefix}elbow_motor">
+      <actuator name="${prefix}joint_3_motor">
         <mechanicalReduction>1</mechanicalReduction>
       </actuator>
     </transmission>
-    <transmission name="${prefix}wrist_1_trans">
+    <transmission name="${prefix}joint_4_trans">
       <type>transmission_interface/SimpleTransmission</type>
-      <joint name="${prefix}wrist_1_joint">
+      <joint name="${prefix}joint_4">
         <hardwareInterface>${hw_interface}</hardwareInterface>
       </joint>
-      <actuator name="${prefix}wrist_1_motor">
+      <actuator name="${prefix}joint_4_motor">
         <mechanicalReduction>1</mechanicalReduction>
       </actuator>
     </transmission>
-    <transmission name="${prefix}wrist_2_trans">
+    <transmission name="${prefix}joint_5_trans">
       <type>transmission_interface/SimpleTransmission</type>
-      <joint name="${prefix}wrist_2_joint">
+      <joint name="${prefix}joint_5">
         <hardwareInterface>${hw_interface}</hardwareInterface>
       </joint>
-      <actuator name="${prefix}wrist_2_motor">
+      <actuator name="${prefix}joint_5_motor">
         <mechanicalReduction>1</mechanicalReduction>
       </actuator>
     </transmission>
-    <transmission name="${prefix}wrist_3_trans">
+    <transmission name="${prefix}joint_6_trans">
       <type>transmission_interface/SimpleTransmission</type>
-      <joint name="${prefix}wrist_3_joint">
+      <joint name="${prefix}joint_6">
         <hardwareInterface>${hw_interface}</hardwareInterface>
       </joint>
-      <actuator name="${prefix}wrist_3_motor">
+      <actuator name="${prefix}joint_6_motor">
         <mechanicalReduction>1</mechanicalReduction>
       </actuator>

File: ur_description/urdf/ur10.urdf.xacro (robot description, xacro)
@@ -81,5 +81,6 @@
       </xacro:cylinder_inertial>
     </link>
-    <joint name="${prefix}shoulder_pan_joint" type="revolute">
+    <!--joint name="${prefix}shoulder_pan_joint" type="revolute"-->
+    <joint name="${prefix}joint_1" type="revolute">
       <parent link="${prefix}base_link" />
       <child link = "${prefix}shoulder_link" />
@@ -118,5 +119,6 @@
       </xacro:cylinder_inertial>
     </link>
-    <joint name="${prefix}shoulder_lift_joint" type="revolute">
+    <!--joint name="${prefix}shoulder_lift_joint" type="revolute"-->
+    <joint name="${prefix}joint_2" type="revolute">
       <parent link="${prefix}shoulder_link" />
       <child link = "${prefix}upper_arm_link" />
@@ -155,5 +157,6 @@
       </xacro:cylinder_inertial>
     </link>
-    <joint name="${prefix}elbow_joint" type="revolute">
+    <!--joint name="${prefix}elbow_joint" type="revolute"-->
+    <joint name="${prefix}joint_3" type="revolute">
       <parent link="${prefix}upper_arm_link" />
       <child link = "${prefix}forearm_link" />
@@ -192,5 +195,6 @@
       </xacro:cylinder_inertial>
     </link>
-    <joint name="${prefix}wrist_1_joint" type="revolute">
+    <!--joint name="${prefix}wrist_1_joint" type="revolute"-->
+    <joint name="${prefix}joint_4" type="revolute">
       <parent link="${prefix}forearm_link" />
       <child link = "${prefix}wrist_1_link" />
@@ -229,5 +233,6 @@
       </xacro:cylinder_inertial>
     </link>
-    <joint name="${prefix}wrist_2_joint" type="revolute">
+    <!--joint name="${prefix}wrist_2_joint" type="revolute"-->
+    <joint name="${prefix}joint_5" type="revolute">
       <parent link="${prefix}wrist_1_link" />
       <child link = "${prefix}wrist_2_link" />
@@ -266,5 +271,6 @@
       </xacro:cylinder_inertial>
     </link>
-    <joint name="${prefix}wrist_3_joint" type="revolute">
+    <!--joint name="${prefix}wrist_3_joint" type="revolute"-->
+    <joint name="${prefix}joint_6" type="revolute">
       <parent link="${prefix}wrist_2_link" />
       <child link = "${prefix}wrist_3_link" />
