Commit message: rename joints

File: ur_description/urdf/ur.transmission.xacro (robot description, xacro)
@@ -2,61 +2,61 @@
 <robot xmlns:xacro="http://ros.org/wiki/xacro">
   <xacro:macro name="ur_arm_transmission" params="prefix">
-    <transmission name="${prefix}shoulder_pan_trans">
+    <transmission name="${prefix}1_trans">
       <type>transmission_interface/SimpleTransmission</type>
-      <joint name="${prefix}shoulder_pan_joint">
+      <joint name="${prefix}1_joint">
         <hardwareInterface>PositionJointInterface</hardwareInterface>
         <hardwareInterface>VelocityJointInterface</hardwareInterface>
       </joint>
-      <actuator name="${prefix}shoulder_pan_motor">
+      <actuator name="${prefix}1_motor">
         <mechanicalReduction>1</mechanicalReduction>
       </actuator>
     </transmission>
-    <transmission name="${prefix}shoulder_lift_trans">
+    <transmission name="${prefix}2_trans">
       <type>transmission_interface/SimpleTransmission</type>
-      <joint name="${prefix}shoulder_lift_joint">
+      <joint name="${prefix}2_joint">
         <hardwareInterface>PositionJointInterface</hardwareInterface>
         <hardwareInterface>VelocityJointInterface</hardwareInterface>
       </joint>
-      <actuator name="${prefix}shoulder_lift_motor">
+      <actuator name="${prefix}2_motor">
         <mechanicalReduction>1</mechanicalReduction>
       </actuator>
     </transmission>
-    <transmission name="${prefix}elbow_trans">
+    <transmission name="${prefix}3_trans">
       <type>transmission_interface/SimpleTransmission</type>
-      <joint name="${prefix}elbow_joint">
+      <joint name="${prefix}3_joint">
         <hardwareInterface>PositionJointInterface</hardwareInterface>
         <hardwareInterface>VelocityJointInterface</hardwareInterface>
       </joint>
-      <actuator name="${prefix}elbow_motor">
+      <actuator name="${prefix}3_motor">
         <mechanicalReduction>1</mechanicalReduction>
       </actuator>
     </transmission>
-    <transmission name="${prefix}wrist_1_trans">
+    <transmission name="${prefix}4_trans">
       <type>transmission_interface/SimpleTransmission</type>
-      <joint name="${prefix}wrist_1_joint">
+      <joint name="${prefix}4_joint">
         <hardwareInterface>PositionJointInterface</hardwareInterface>
         <hardwareInterface>VelocityJointInterface</hardwareInterface>
       </joint>
-      <actuator name="${prefix}wrist_1_motor">
+      <actuator name="${prefix}4_motor">
         <mechanicalReduction>1</mechanicalReduction>
       </actuator>
     </transmission>
-    <transmission name="${prefix}wrist_2_trans">
+    <transmission name="${prefix}5_trans">
       <type>transmission_interface/SimpleTransmission</type>
-      <joint name="${prefix}wrist_2_joint">
+      <joint name="${prefix}5_joint">
         <hardwareInterface>PositionJointInterface</hardwareInterface>
         <hardwareInterface>VelocityJointInterface</hardwareInterface>
       </joint>
-      <actuator name="${prefix}wrist_2_motor">
+      <actuator name="${prefix}5_motor">
         <mechanicalReduction>1</mechanicalReduction>
       </actuator>
     </transmission>
-    <transmission name="${prefix}wrist_3_trans">
+    <transmission name="${prefix}6_trans">
       <type>transmission_interface/SimpleTransmission</type>
-      <joint name="${prefix}wrist_3_joint">
+      <joint name="${prefix}6_joint">
         <hardwareInterface>PositionJointInterface</hardwareInterface>
         <hardwareInterface>VelocityJointInterface</hardwareInterface>
       </joint>
-      <actuator name="${prefix}wrist_3_motor">
+      <actuator name="${prefix}6_motor">
         <mechanicalReduction>1</mechanicalReduction>
       </actuator>

File: ur_description/urdf/ur10.urdf.xacro (robot description, xacro)
@@ -78,5 +78,5 @@
       </xacro:cylinder_inertial>
     </link>
-    <joint name="${prefix}shoulder_pan_joint" type="revolute">
+    <joint name="${prefix}1_joint" type="revolute">
       <parent link="${prefix}base_link" />
       <child link = "${prefix}shoulder_link" />
@@ -109,5 +109,5 @@
       </xacro:cylinder_inertial>
     </link>
-    <joint name="${prefix}shoulder_lift_joint" type="revolute">
+    <joint name="${prefix}2_joint" type="revolute">
       <parent link="${prefix}shoulder_link" />
       <child link = "${prefix}upper_arm_link" />
@@ -140,5 +140,5 @@
       </xacro:cylinder_inertial>
     </link>
-    <joint name="${prefix}elbow_joint" type="revolute">
+    <joint name="${prefix}3_joint" type="revolute">
       <parent link="${prefix}upper_arm_link" />
       <child link = "${prefix}forearm_link" />
@@ -171,5 +171,5 @@
       </xacro:cylinder_inertial>
     </link>
-    <joint name="${prefix}wrist_1_joint" type="revolute">
+    <joint name="${prefix}4_joint" type="revolute">
       <parent link="${prefix}forearm_link" />
       <child link = "${prefix}wrist_1_link" />
@@ -202,5 +202,5 @@
       </xacro:cylinder_inertial>
     </link>
-    <joint name="${prefix}wrist_2_joint" type="revolute">
+    <joint name="${prefix}5_joint" type="revolute">
       <parent link="${prefix}wrist_1_link" />
       <child link = "${prefix}wrist_2_link" />
@@ -233,5 +233,5 @@
       </xacro:cylinder_inertial>
     </link>
-    <joint name="${prefix}wrist_3_joint" type="revolute">
+    <joint name="${prefix}6_joint" type="revolute">
       <parent link="${prefix}wrist_2_link" />
       <child link = "${prefix}wrist_3_link" />

Commit message: undo robot names

File: ur_description/urdf/ur.transmission.xacro (robot description, xacro)
@@ -2,61 +2,61 @@
 <robot xmlns:xacro="http://ros.org/wiki/xacro">
   <xacro:macro name="ur_arm_transmission" params="prefix">
-    <transmission name="${prefix}1_trans">
+    <transmission name="${prefix}shoulder_pan_trans">
       <type>transmission_interface/SimpleTransmission</type>
-      <joint name="${prefix}1_joint">
+      <joint name="${prefix}shoulder_pan_joint">
         <hardwareInterface>PositionJointInterface</hardwareInterface>
         <hardwareInterface>VelocityJointInterface</hardwareInterface>
       </joint>
-      <actuator name="${prefix}1_motor">
+      <actuator name="${prefix}shoulder_pan_motor">
         <mechanicalReduction>1</mechanicalReduction>
       </actuator>
     </transmission>
-    <transmission name="${prefix}2_trans">
+    <transmission name="${prefix}shoulder_lift_trans">
       <type>transmission_interface/SimpleTransmission</type>
-      <joint name="${prefix}2_joint">
+      <joint name="${prefix}shoulder_lift_joint">
         <hardwareInterface>PositionJointInterface</hardwareInterface>
         <hardwareInterface>VelocityJointInterface</hardwareInterface>
       </joint>
-      <actuator name="${prefix}2_motor">
+      <actuator name="${prefix}shoulder_lift_motor">
         <mechanicalReduction>1</mechanicalReduction>
       </actuator>
     </transmission>
-    <transmission name="${prefix}3_trans">
+    <transmission name="${prefix}elbow_trans">
       <type>transmission_interface/SimpleTransmission</type>
-      <joint name="${prefix}3_joint">
+      <joint name="${prefix}elbow_joint">
         <hardwareInterface>PositionJointInterface</hardwareInterface>
         <hardwareInterface>VelocityJointInterface</hardwareInterface>
       </joint>
-      <actuator name="${prefix}3_motor">
+      <actuator name="${prefix}elbow_motor">
         <mechanicalReduction>1</mechanicalReduction>
       </actuator>
     </transmission>
-    <transmission name="${prefix}4_trans">
+    <transmission name="${prefix}wrist_1_trans">
       <type>transmission_interface/SimpleTransmission</type>
-      <joint name="${prefix}4_joint">
+      <joint name="${prefix}wrist_1_joint">
         <hardwareInterface>PositionJointInterface</hardwareInterface>
         <hardwareInterface>VelocityJointInterface</hardwareInterface>
       </joint>
-      <actuator name="${prefix}4_motor">
+      <actuator name="${prefix}wrist_1_motor">
         <mechanicalReduction>1</mechanicalReduction>
       </actuator>
     </transmission>
-    <transmission name="${prefix}5_trans">
+    <transmission name="${prefix}wrist_2_trans">
       <type>transmission_interface/SimpleTransmission</type>
-      <joint name="${prefix}5_joint">
+      <joint name="${prefix}wrist_2_joint">
         <hardwareInterface>PositionJointInterface</hardwareInterface>
         <hardwareInterface>VelocityJointInterface</hardwareInterface>
       </joint>
-      <actuator name="${prefix}5_motor">
+      <actuator name="${prefix}wrist_2_motor">
         <mechanicalReduction>1</mechanicalReduction>
       </actuator>
     </transmission>
-    <transmission name="${prefix}6_trans">
+    <transmission name="${prefix}wrist_elbow_trans">
       <type>transmission_interface/SimpleTransmission</type>
-      <joint name="${prefix}6_joint">
+      <joint name="${prefix}wrist_elbow_joint">
         <hardwareInterface>PositionJointInterface</hardwareInterface>
         <hardwareInterface>VelocityJointInterface</hardwareInterface>
       </joint>
-      <actuator name="${prefix}6_motor">
+      <actuator name="${prefix}wrist_elbow_motor">
         <mechanicalReduction>1</mechanicalReduction>
       </actuator>

File: ur_description/urdf/ur10.urdf.xacro (robot description, xacro)
@@ -78,7 +78,7 @@
       </xacro:cylinder_inertial>
     </link>
-    <joint name="${prefix}1_joint" type="revolute">
+    <joint name="${prefix}shoulder_pan_joint" type="revolute">
       <parent link="${prefix}base_link" />
-      <child link = "${prefix}1_link" />
+      <child link = "${prefix}shoulder_pan_link" />
       <origin xyz="0.0 0.0 ${shoulder_height}" rpy="0.0 0.0 0.0" />
       <axis xyz="0 0 1" />
@@ -91,5 +91,5 @@
       <dynamics damping="0.0" friction="0.0"/>
     </joint>
-    <link name="${prefix}1_link">
+    <link name="${prefix}shoulder_pan_link">
       <visual>
         <geometry>
@@ -109,7 +109,7 @@
       </xacro:cylinder_inertial>
     </link>
-    <joint name="${prefix}2_joint" type="revolute">
-      <parent link="${prefix}1_link" />
-      <child link = "${prefix}2_link" />
+    <joint name="${prefix}shoulder_lift_joint" type="revolute">
+      <parent link="${prefix}shoulder_pan_link" />
+      <child link = "${prefix}shoulder_lift_link" />
       <origin xyz="0.0 ${shoulder_offset} 0.0" rpy="0.0 ${pi / 2.0} 0.0" />
       <axis xyz="0 1 0" />
@@ -122,5 +122,5 @@
       <dynamics damping="0.0" friction="0.0"/>
     </joint>
-    <link name="${prefix}2_link">
+    <link name="${prefix}shoulder_lift_link">
       <visual>
         <geometry>
@@ -140,7 +140,7 @@
       </xacro:cylinder_inertial>
     </link>
-    <joint name="${prefix}3_joint" type="revolute">
-      <parent link="${prefix}2_link" />
-      <child link = "${prefix}3_link" />
+    <joint name="${prefix}elbow_joint" type="revolute">
+      <parent link="${prefix}shoulder_lift_link" />
+      <child link = "${prefix}elbow_link" />
       <origin xyz="0.0 ${elbow_offset} ${upper_arm_length}" rpy="0.0 0.0 0.0" />
       <axis xyz="0 1 0" />
@@ -153,5 +153,5 @@
       <dynamics damping="0.0" friction="0.0"/>
     </joint>
-    <link name="${prefix}3_link">
+    <link name="${prefix}elbow_link">
       <visual>
          <geometry>
@@ -171,7 +171,7 @@
       </xacro:cylinder_inertial>
     </link>
-    <joint name="${prefix}4_joint" type="revolute">
-      <parent link="${prefix}3_link" />
-      <child link = "${prefix}4_link" />
+    <joint name="${prefix}wrist_1_joint" type="revolute">
+      <parent link="${prefix}elbow_link" />
+      <child link = "${prefix}wrist_1_link" />
       <origin xyz="0.0 0.0 ${forearm_length}" rpy="0.0 ${pi / 2.0} 0.0" />
       <axis xyz="0 1 0" />
@@ -184,5 +184,5 @@
       <dynamics damping="0.0" friction="0.0"/>
     </joint>
-    <link name="${prefix}4_link">
+    <link name="${prefix}wrist_1_link">
       <visual>
         <geometry>
@@ -202,7 +202,7 @@
       </xacro:cylinder_inertial>
     </link>
-    <joint name="${prefix}5_joint" type="revolute">
-      <parent link="${prefix}4_link" />
-      <child link = "${prefix}5_link" />
+    <joint name="${prefix}wrist_2_joint" type="revolute">
+      <parent link="${prefix}wrist_1_link" />
+      <child link = "${prefix}wrist_2_link" />
       <origin xyz="0.0 ${wrist_1_length} 0.0" rpy="0.0 0.0 0.0" />
       <axis xyz="0 0 1" />
@@ -215,5 +215,5 @@
       <dynamics damping="0.0" friction="0.0"/>
     </joint>
-    <link name="${prefix}5_link">
+    <link name="${prefix}wrist_2_link">
       <visual>
         <geometry>
@@ -233,7 +233,7 @@
       </xacro:cylinder_inertial>
     </link>
-    <joint name="${prefix}6_joint" type="revolute">
-      <parent link="${prefix}5_link" />
-      <child link = "${prefix}6_link" />
+    <joint name="${prefix}wrist_3_joint" type="revolute">
+      <parent link="${prefix}wrist_2_link" />
+      <child link = "${prefix}wrist_3_link" />
       <origin xyz="0.0 0.0 ${wrist_2_length}" rpy="0.0 0.0 0.0" />
       <axis xyz="0 1 0" />
@@ -246,5 +246,5 @@
       <dynamics damping="0.0" friction="0.0"/>
     </joint>
-    <link name="${prefix}6_link">
+    <link name="${prefix}wrist_3_link">
       <visual>
         <geometry>
@@ -265,5 +265,5 @@
     </link>
     <joint name="${prefix}ee_fixed_joint" type="fixed">
-      <parent link="${prefix}6_link" />
+      <parent link="${prefix}wrist_3_link" />
       <child link = "${prefix}ee_link" />
       <origin xyz="0.0 ${wrist_3_length} 0.0" rpy="0.0 0.0 ${pi/2.0}" />
@@ -301,5 +301,5 @@
     <joint name="${prefix}wrist_3_link-tool0_fixed_joint" type="fixed">
       <origin xyz="0.0 ${wrist_3_length+0.14} 0.0" rpy="0.0 0.0 ${pi/2.0}" />
-      <parent link="${prefix}6_link"/>
+      <parent link="${prefix}wrist_3_link"/>
       <child link="${prefix}tool0"/>
       <xacro:unless value="${joint_limited}">

File: ur_description/urdf/ur10_joint_limited_robot.urdf.xacro (robot description, xacro)
@@ -6,18 +6,41 @@
   <!-- ur10 -->
   <xacro:include filename="$(find ur_description)/urdf/ur10.urdf.xacro" />
+ <link name="world" />
+ <joint name="world-robot_base_joint" type="fixed">
+   <origin xyz="-0.50 -0.30 0.30" rpy="0 0 0" />
+   <parent link="world"/>
+   <child link="robot_base"/>
+ </joint>
+ <link name="robot_base">
+     <visual>
+       <origin rpy="0 0 0" xyz="0 0 0"/>
+       <geometry>
+         <box size="1.0 0.60 0.60"/>
+       </geometry>
+       <material name="LightGrey">
+         <color rgba="0.7 0.7 0.7 1.0"/>
+       </material>
+     </visual>
+ </link>
+ <joint name="world_joint" type="fixed">
+   <parent link="robot_base" />
+   <child link = "base_link" />
+   <origin xyz="0.324 -0.191 0.2925" rpy="0.0 0.0 -2.3562" />
+ </joint>
   <!-- arm -->
   <xacro:ur10_robot prefix="" joint_limited="true"
-		 shoulder_pan_lower_limit="${-pi}" shoulder_pan_upper_limit="${pi}"
-		 shoulder_lift_lower_limit="${-pi}" shoulder_lift_upper_limit="${pi}"
-		 elbow_joint_lower_limit="${-pi}" elbow_joint_upper_limit="${pi}"
-		 wrist_1_lower_limit="${-pi}" wrist_1_upper_limit="${pi}"
-		 wrist_2_lower_limit="${-pi}" wrist_2_upper_limit="${pi}"
-		 wrist_3_lower_limit="${-pi}" wrist_3_upper_limit="${pi}"
-/>
-  <link name="world" />
-  <joint name="world_joint" type="fixed">
-    <parent link="world" />
-    <child link = "base_link" />
-    <origin xyz="0.0 0.0 0.0" rpy="0.0 0.0 0.0" />
-  </joint>
+               shoulder_pan_lower_limit="${-pi}" shoulder_pan_upper_limit="${pi}"
+               shoulder_lift_lower_limit="${-pi}" shoulder_lift_upper_limit="${pi}"
+               elbow_joint_lower_limit="${-pi}" elbow_joint_upper_limit="${pi}"
+               wrist_1_lower_limit="${-pi}" wrist_1_upper_limit="${pi}"
+               wrist_2_lower_limit="${-pi}" wrist_2_upper_limit="${pi}"
+               wrist_3_lower_limit="${-pi}" wrist_3_upper_limit="${pi}"
+  />
+  <!-- ros_control plugin -->
+  <gazebo>
+    <plugin name="ros_control" filename="libhwi_switch_gazebo_ros_control.so">
+      <robotNamespace></robotNamespace>
+      <filterJointsParam>joint_names</filterJointsParam>
+    </plugin>
+  </gazebo>
 </robot>

File: ur_description/urdf/ur10_robot.urdf.xacro (robot description, xacro)
@@ -31,13 +31,13 @@
   <joint name="world_joint" type="fixed">
     <parent link="robot_base" />
-    <child link = "arm_base_link" />
+    <child link = "base_link" />
     <origin xyz="0.324 -0.191 0.2925" rpy="0.0 0.0 -2.3562" />
   </joint>
   <!-- arm -->
-  <xacro:ur10_robot prefix="arm_" joint_limited="false"/>
+  <xacro:ur10_robot prefix="" joint_limited="false"/>
   <!-- ros_control plugin -->
   <gazebo>
     <plugin name="ros_control" filename="libhwi_switch_gazebo_ros_control.so">
-      <robotNamespace>arm</robotNamespace>
+      <robotNamespace></robotNamespace>
       <filterJointsParam>joint_names</filterJointsParam>
     </plugin>

Commit message: correct naming

File: ur_description/urdf/ur.transmission.xacro (robot description, xacro)
@@ -52,11 +52,11 @@
       </actuator>
     </transmission>
-    <transmission name="${prefix}wrist_elbow_trans">
+    <transmission name="${prefix}wrist_3_trans">
       <type>transmission_interface/SimpleTransmission</type>
-      <joint name="${prefix}wrist_elbow_joint">
+      <joint name="${prefix}wrist_3_joint">
         <hardwareInterface>PositionJointInterface</hardwareInterface>
         <hardwareInterface>VelocityJointInterface</hardwareInterface>
       </joint>
-      <actuator name="${prefix}wrist_elbow_motor">
+      <actuator name="${prefix}wrist_3_motor">
         <mechanicalReduction>1</mechanicalReduction>
       </actuator>
