Commit message: rename joints and remove prefix

File: ur_description/urdf/ur.transmission.xacro (robot description, xacro)
@@ -2,61 +2,61 @@
 <robot xmlns:xacro="http://ros.org/wiki/xacro">
   <xacro:macro name="ur_arm_transmission" params="prefix">
-    <transmission name="${prefix}1_trans">
+    <transmission name="${prefix}shoulder_1_trans">
       <type>transmission_interface/SimpleTransmission</type>
-      <joint name="${prefix}1_joint">
+      <joint name="${prefix}shoulder_1_joint">
         <hardwareInterface>PositionJointInterface</hardwareInterface>
         <hardwareInterface>VelocityJointInterface</hardwareInterface>
       </joint>
-      <actuator name="${prefix}1_motor">
+      <actuator name="${prefix}shoulder_1_motor">
         <mechanicalReduction>1</mechanicalReduction>
       </actuator>
     </transmission>
-    <transmission name="${prefix}2_trans">
+    <transmission name="${prefix}shoulder_2_trans">
       <type>transmission_interface/SimpleTransmission</type>
-      <joint name="${prefix}2_joint">
+      <joint name="${prefix}shoulder_2_joint">
         <hardwareInterface>PositionJointInterface</hardwareInterface>
         <hardwareInterface>VelocityJointInterface</hardwareInterface>
       </joint>
-      <actuator name="${prefix}2_motor">
+      <actuator name="${prefix}shoulder_2_motor">
         <mechanicalReduction>1</mechanicalReduction>
       </actuator>
     </transmission>
-    <transmission name="${prefix}3_trans">
+    <transmission name="${prefix}shoulder_3_trans">
       <type>transmission_interface/SimpleTransmission</type>
-      <joint name="${prefix}3_joint">
+      <joint name="${prefix}shoulder_3_joint">
         <hardwareInterface>PositionJointInterface</hardwareInterface>
         <hardwareInterface>VelocityJointInterface</hardwareInterface>
       </joint>
-      <actuator name="${prefix}3_motor">
+      <actuator name="${prefix}shoulder_3_motor">
         <mechanicalReduction>1</mechanicalReduction>
       </actuator>
     </transmission>
-    <transmission name="${prefix}4_trans">
+    <transmission name="${prefix}wrist_1_trans">
       <type>transmission_interface/SimpleTransmission</type>
-      <joint name="${prefix}4_joint">
+      <joint name="${prefix}wrist_1_joint">
         <hardwareInterface>PositionJointInterface</hardwareInterface>
         <hardwareInterface>VelocityJointInterface</hardwareInterface>
       </joint>
-      <actuator name="${prefix}4_motor">
+      <actuator name="${prefix}wrist_1_motor">
         <mechanicalReduction>1</mechanicalReduction>
       </actuator>
     </transmission>
-    <transmission name="${prefix}5_trans">
+    <transmission name="${prefix}wrist_2_trans">
       <type>transmission_interface/SimpleTransmission</type>
-      <joint name="${prefix}5_joint">
+      <joint name="${prefix}wrist_2_joint">
         <hardwareInterface>PositionJointInterface</hardwareInterface>
         <hardwareInterface>VelocityJointInterface</hardwareInterface>
       </joint>
-      <actuator name="${prefix}5_motor">
+      <actuator name="${prefix}wrist_2_motor">
         <mechanicalReduction>1</mechanicalReduction>
       </actuator>
     </transmission>
-    <transmission name="${prefix}6_trans">
+    <transmission name="${prefix}wrist_3_trans">
       <type>transmission_interface/SimpleTransmission</type>
-      <joint name="${prefix}6_joint">
+      <joint name="${prefix}wrist_3_joint">
         <hardwareInterface>PositionJointInterface</hardwareInterface>
         <hardwareInterface>VelocityJointInterface</hardwareInterface>
       </joint>
-      <actuator name="${prefix}6_motor">
+      <actuator name="${prefix}wrist_3_motor">
         <mechanicalReduction>1</mechanicalReduction>
       </actuator>

File: ur_description/urdf/ur10.urdf.xacro (robot description, xacro)
@@ -78,5 +78,5 @@
       </xacro:cylinder_inertial>
     </link>
-    <joint name="${prefix}1_joint" type="revolute">
+    <joint name="${prefix}shoulder_1_joint" type="revolute">
       <parent link="${prefix}base_link" />
       <child link = "${prefix}shoulder_pan_link" />
@@ -109,5 +109,5 @@
       </xacro:cylinder_inertial>
     </link>
-    <joint name="${prefix}2_joint" type="revolute">
+    <joint name="${prefix}shoulder_2_joint" type="revolute">
       <parent link="${prefix}shoulder_pan_link" />
       <child link = "${prefix}shoulder_lift_link" />
@@ -140,5 +140,5 @@
       </xacro:cylinder_inertial>
     </link>
-    <joint name="${prefix}3_joint" type="revolute">
+    <joint name="${prefix}shoulder_3_joint" type="revolute">
       <parent link="${prefix}shoulder_lift_link" />
       <child link = "${prefix}elbow_link" />
@@ -171,5 +171,5 @@
       </xacro:cylinder_inertial>
     </link>
-    <joint name="${prefix}4_joint" type="revolute">
+    <joint name="${prefix}wrist_1_joint" type="revolute">
       <parent link="${prefix}elbow_link" />
       <child link = "${prefix}wrist_1_link" />
@@ -202,5 +202,5 @@
       </xacro:cylinder_inertial>
     </link>
-    <joint name="${prefix}5_joint" type="revolute">
+    <joint name="${prefix}wrist_2_joint" type="revolute">
       <parent link="${prefix}wrist_1_link" />
       <child link = "${prefix}wrist_2_link" />
@@ -233,5 +233,5 @@
       </xacro:cylinder_inertial>
     </link>
-    <joint name="${prefix}6_joint" type="revolute">
+    <joint name="${prefix}wrist_3_joint" type="revolute">
       <parent link="${prefix}wrist_2_link" />
       <child link = "${prefix}wrist_3_link" />

File: ur_description/urdf/ur10_joint_limited_robot.urdf.xacro (robot description, xacro)
@@ -34,9 +34,9 @@
     <joint name="world_joint" type="fixed">
       <parent link="robot_base" />
-      <child link = "arm_base_link" />
+      <child link = "base_link" />
       <origin xyz="0.0 0.0 0.45" rpy="0.0 0.0 -2.3562" />
     </joint>
   <!-- arm -->
-  <xacro:ur10_robot prefix="arm_" joint_limited="true"
+  <xacro:ur10_robot prefix="" joint_limited="true"
                shoulder_pan_lower_limit="${-pi}" shoulder_pan_upper_limit="${pi}"
                shoulder_lift_lower_limit="${-pi}" shoulder_lift_upper_limit="${pi}"
@@ -49,6 +49,6 @@
   <gazebo>
     <plugin name="ros_control" filename="libhwi_switch_gazebo_ros_control.so">
-      <robotNamespace>arm</robotNamespace>
-      <filterJointsParam>joint_names</filterJointsParam>
+      <!--robotNamespace>arm</robotNamespace>
+      <filterJointsParam>joint_names</filterJointsParam-->
     </plugin>
   </gazebo>

File: ur_description/urdf/ur10_robot.urdf.xacro (robot description, xacro)
@@ -34,14 +34,14 @@
   <joint name="world_joint" type="fixed">
     <parent link="robot_base" />
-    <child link = "arm_base_link" />
+    <child link = "base_link" />
     <origin xyz="0.0 0.0 0.45" rpy="0.0 0.0 -2.3562" />
   </joint>
   <!-- arm -->
-  <xacro:ur10_robot prefix="arm_" joint_limited="false"/>
+  <xacro:ur10_robot prefix="" joint_limited="false"/>
   <!-- ros_control plugin -->
   <gazebo>
     <plugin name="ros_control" filename="libhwi_switch_gazebo_ros_control.so">
-      <robotNamespace>arm</robotNamespace>
-      <filterJointsParam>joint_names</filterJointsParam>
+      <!--robotNamespace>arm</robotNamespace>
+      <filterJointsParam>joint_names</filterJointsParam-->
     </plugin>
   </gazebo>

Commit message: add cob control

File: ur_description/urdf/ur.transmission.xacro (robot description, xacro)
@@ -5,6 +5,6 @@
       <type>transmission_interface/SimpleTransmission</type>
       <joint name="${prefix}1_joint">
-        <hardwareInterface>PositionJointInterface</hardwareInterface>
-        <hardwareInterface>VelocityJointInterface</hardwareInterface>
+        <hardwareInterface>hardware_interface/PositionJointInterface</hardwareInterface>
+        <hardwareInterface>hardware_interface/VelocityJointInterface</hardwareInterface>
       </joint>
       <actuator name="${prefix}1_motor">
@@ -15,6 +15,6 @@
       <type>transmission_interface/SimpleTransmission</type>
       <joint name="${prefix}2_joint">
-        <hardwareInterface>PositionJointInterface</hardwareInterface>
-        <hardwareInterface>VelocityJointInterface</hardwareInterface>
+        <hardwareInterface>hardware_interface/PositionJointInterface</hardwareInterface>
+        <hardwareInterface>hardware_interface/VelocityJointInterface</hardwareInterface>
       </joint>
       <actuator name="${prefix}2_motor">
@@ -25,6 +25,6 @@
       <type>transmission_interface/SimpleTransmission</type>
       <joint name="${prefix}3_joint">
-        <hardwareInterface>PositionJointInterface</hardwareInterface>
-        <hardwareInterface>VelocityJointInterface</hardwareInterface>
+        <hardwareInterface>hardware_interface/PositionJointInterface</hardwareInterface>
+        <hardwareInterface>hardware_interface/VelocityJointInterface</hardwareInterface>
       </joint>
       <actuator name="${prefix}3_motor">
@@ -35,6 +35,6 @@
       <type>transmission_interface/SimpleTransmission</type>
       <joint name="${prefix}4_joint">
-        <hardwareInterface>PositionJointInterface</hardwareInterface>
-        <hardwareInterface>VelocityJointInterface</hardwareInterface>
+        <hardwareInterface>hardware_interface/PositionJointInterface</hardwareInterface>
+        <hardwareInterface>hardware_interface/VelocityJointInterface</hardwareInterface>
       </joint>
       <actuator name="${prefix}4_motor">
@@ -45,6 +45,6 @@
       <type>transmission_interface/SimpleTransmission</type>
       <joint name="${prefix}5_joint">
-        <hardwareInterface>PositionJointInterface</hardwareInterface>
-        <hardwareInterface>VelocityJointInterface</hardwareInterface>
+        <hardwareInterface>hardware_interface/PositionJointInterface</hardwareInterface>
+        <hardwareInterface>hardware_interface/VelocityJointInterface</hardwareInterface>
       </joint>
       <actuator name="${prefix}5_motor">
@@ -55,6 +55,6 @@
       <type>transmission_interface/SimpleTransmission</type>
       <joint name="${prefix}6_joint">
-        <hardwareInterface>PositionJointInterface</hardwareInterface>
-        <hardwareInterface>VelocityJointInterface</hardwareInterface>
+        <hardwareInterface>hardware_interface/PositionJointInterface</hardwareInterface>
+        <hardwareInterface>hardware_interface/VelocityJointInterface</hardwareInterface>
       </joint>
       <actuator name="${prefix}6_motor">
@@ -65,6 +65,6 @@
       <type>transmission_interface/SimpleTransmission</type>
       <joint name="${prefix}ee_fixed_joint">
-        <hardwareInterface>PositionJointInterface</hardwareInterface>
-        <hardwareInterface>VelocityJointInterface</hardwareInterface>
+        <hardwareInterface>hardware_interface/PositionJointInterface</hardwareInterface>
+        <hardwareInterface>hardware_interface/VelocityJointInterface</hardwareInterface>
       </joint>
       <actuator name="${prefix}ee_fixed_motor">

File: ur_description/urdf/ur10_robot.urdf.xacro (robot description, xacro)
@@ -10,5 +10,5 @@
     <parent link="world" />
     <child link = "arm_base_link" />
-    <origin xyz="0.0 0.0 0.0" rpy="0.0 0.0 0.0" />
+    <origin xyz="-0.50 -0.30 0.30" rpy="0.0 0.0 0.0" />
   </joint>
  <!--
@@ -40,7 +40,8 @@
   <!-- ros_control plugin -->
   <gazebo>
-    <plugin name="ros_control" filename="libhwi_switch_gazebo_ros_control.so">
+    <plugin name="gazebo_ros_control" filename="libhwi_switch_gazebo_ros_control.so">
       <robotNamespace>arm</robotNamespace>
       <filterJointsParam>joint_names</filterJointsParam>
+      <robotSimType>cob_gazebo_ros_control/HWISwitchRobotHWSim</robotSimType>
     </plugin>
   </gazebo>
