Commit message: add prefix

File: ur_description/urdf/ur10_joint_limited_robot.urdf.xacro (robot description, xacro)
@@ -6,18 +6,47 @@
   <!-- ur10 -->
   <xacro:include filename="$(find ur_description)/urdf/ur10.urdf.xacro" />
-  <!-- arm -->
-  <xacro:ur10_robot prefix="" joint_limited="true"
-		 shoulder_pan_lower_limit="${-pi}" shoulder_pan_upper_limit="${pi}"
-		 shoulder_lift_lower_limit="${-pi}" shoulder_lift_upper_limit="${pi}"
-		 elbow_joint_lower_limit="${-pi}" elbow_joint_upper_limit="${pi}"
-		 wrist_1_lower_limit="${-pi}" wrist_1_upper_limit="${pi}"
-		 wrist_2_lower_limit="${-pi}" wrist_2_upper_limit="${pi}"
-		 wrist_3_lower_limit="${-pi}" wrist_3_upper_limit="${pi}"
-/>
-  <link name="world" />
+  <!--link name="world" />
   <joint name="world_joint" type="fixed">
     <parent link="world" />
     <child link = "base_link" />
     <origin xyz="0.0 0.0 0.0" rpy="0.0 0.0 0.0" />
-  </joint>
+  </joint-->
+    <link name="world" />
+    <joint name="world-robot_base_joint" type="fixed">
+        <origin xyz="-0.65 -0.45 0.45" rpy="0 0 0" />
+        <parent link="world"/>
+        <child link="robot_base"/>
+    </joint>
+    <link name="robot_base">
+        <visual>
+            <origin rpy="0 0 0" xyz="0 0 0"/>
+            <geometry>
+                <box size="1.30 0.90 0.90"/>
+            </geometry>
+            <material name="LightGrey">
+                <color rgba="0.7 0.7 0.7 1.0"/>
+            </material>
+        </visual>
+    </link>
+    <joint name="world_joint" type="fixed">
+        <parent link="robot_base" />
+        <child link = "arm_base_link" />
+        <origin xyz="0.324 -0.191 0.2925" rpy="0.0 0.0 -2.3562" />
+    </joint>
+    <!-- arm -->
+    <xacro:ur10_robot prefix="arm_" joint_limited="true"
+                   shoulder_pan_lower_limit="${-pi}" shoulder_pan_upper_limit="${pi}"
+                   shoulder_lift_lower_limit="${-pi}" shoulder_lift_upper_limit="${pi}"
+                   elbow_joint_lower_limit="${-pi}" elbow_joint_upper_limit="${pi}"
+                   wrist_1_lower_limit="${-pi}" wrist_1_upper_limit="${pi}"
+                   wrist_2_lower_limit="${-pi}" wrist_2_upper_limit="${pi}"
+                   wrist_3_lower_limit="${-pi}" wrist_3_upper_limit="${pi}"
+    />
+    <!-- ros_control plugin -->
+    <gazebo>
+        <plugin name="ros_control" filename="libhwi_switch_gazebo_ros_control.so">
+            <robotNamespace>arm</robotNamespace>
+            <filterJointsParam>joint_names</filterJointsParam>
+        </plugin>
+    </gazebo>
 </robot>

Commit message: add prefix to arm and change controller joint names

File: ur_description/urdf/ur10_joint_limited_robot.urdf.xacro (robot description, xacro)
@@ -25,9 +25,9 @@
  <joint name="world_joint" type="fixed">
    <parent link="robot_base" />
-   <child link = "base_link" />
+   <child link = "arm_base_link" />
    <origin xyz="0.324 -0.191 0.2925" rpy="0.0 0.0 -2.3562" />
  </joint>
   <!-- arm -->
-  <xacro:ur10_robot prefix="" joint_limited="true"
+  <xacro:ur10_robot prefix="arm_" joint_limited="true"
                shoulder_pan_lower_limit="${-pi}" shoulder_pan_upper_limit="${pi}"
                shoulder_lift_lower_limit="${-pi}" shoulder_lift_upper_limit="${pi}"
@@ -40,5 +40,5 @@
   <gazebo>
     <plugin name="ros_control" filename="libhwi_switch_gazebo_ros_control.so">
-      <robotNamespace></robotNamespace>
+      <robotNamespace>arm</robotNamespace>
       <filterJointsParam>joint_names</filterJointsParam>
     </plugin>

File: ur_description/urdf/ur10_robot.urdf.xacro (robot description, xacro)
@@ -31,13 +31,13 @@
   <joint name="world_joint" type="fixed">
     <parent link="robot_base" />
-    <child link = "base_link" />
+    <child link = "arm_base_link" />
     <origin xyz="0.324 -0.191 0.2925" rpy="0.0 0.0 -2.3562" />
   </joint>
   <!-- arm -->
-  <xacro:ur10_robot prefix="" joint_limited="false"/>
+  <xacro:ur10_robot prefix="arm_" joint_limited="false"/>
   <!-- ros_control plugin -->
   <gazebo>
     <plugin name="ros_control" filename="libhwi_switch_gazebo_ros_control.so">
-      <robotNamespace></robotNamespace>
+      <robotNamespace>arm</robotNamespace>
       <filterJointsParam>joint_names</filterJointsParam>
     </plugin>

Commit message: correct table hegith

File: ur_description/urdf/ur10_joint_limited_robot.urdf.xacro (robot description, xacro)
@@ -6,26 +6,33 @@
   <!-- ur10 -->
   <xacro:include filename="$(find ur_description)/urdf/ur10.urdf.xacro" />
- <link name="world" />
- <joint name="world-robot_base_joint" type="fixed">
-   <origin xyz="-0.50 -0.30 0.30" rpy="0 0 0" />
-   <parent link="world"/>
-   <child link="robot_base"/>
- </joint>
- <link name="robot_base">
-     <visual>
-       <origin rpy="0 0 0" xyz="0 0 0"/>
-       <geometry>
-         <box size="1.0 0.60 0.60"/>
-       </geometry>
-       <material name="LightGrey">
-         <color rgba="0.7 0.7 0.7 1.0"/>
-       </material>
-     </visual>
- </link>
- <joint name="world_joint" type="fixed">
-   <parent link="robot_base" />
-   <child link = "arm_base_link" />
-   <origin xyz="0.324 -0.191 0.2925" rpy="0.0 0.0 -2.3562" />
- </joint>
+    <link name="world" />
+    <joint name="world_joint" type="fixed">
+      <parent link="world" />
+      <child link = "arm_base_link" />
+      <origin xyz="0.0 0.0 0.0" rpy="0.0 0.0 0.0" />
+    </joint>
+    <!-- inlcuding table top robot arm -->
+    <!--link name="world" />
+    <joint name="world-robot_base_joint" type="fixed">
+      <origin xyz="-0.65 -0.45 0.45" rpy="0 0 0" />
+      <parent link="world"/>
+      <child link="robot_base"/>
+    </joint>
+    <link name="robot_base">
+        <visual>
+          <origin rpy="0 0 0" xyz="0 0 0"/>
+          <geometry>
+            <box size="1.30 0.90 0.90"/>
+          </geometry>
+          <material name="LightGrey">
+            <color rgba="0.7 0.7 0.7 1.0"/>
+          </material>
+        </visual>
+    </link>
+    <joint name="world_joint" type="fixed">
+      <parent link="robot_base" />
+      <child link = "arm_base_link" />
+      <origin xyz="0.0 0.0 0.45" rpy="0.0 0.0 -2.3562" />
+    </joint-->
   <!-- arm -->
   <xacro:ur10_robot prefix="arm_" joint_limited="true"

File: ur_description/urdf/ur10_robot.urdf.xacro (robot description, xacro)
@@ -6,13 +6,14 @@
   <!-- ur10 -->
   <xacro:include filename="$(find ur_description)/urdf/ur10.urdf.xacro" />
-  <!--link name="world" />
+  <link name="world" />
   <joint name="world_joint" type="fixed">
     <parent link="world" />
     <child link = "arm_base_link" />
     <origin xyz="0.0 0.0 0.0" rpy="0.0 0.0 0.0" />
-  </joint-->
- <link name="world" />
+  </joint>
+ <!-- inlcuding table top robot arm -->
+ <!--link name="world" />
   <joint name="world-robot_base_joint" type="fixed">
-    <origin xyz="-0.50 -0.30 0.30" rpy="0 0 0" />
+    <origin xyz="-0.65 -0.45 0.45" rpy="0 0 0" />
     <parent link="world"/>
     <child link="robot_base"/>
@@ -22,5 +23,5 @@
         <origin rpy="0 0 0" xyz="0 0 0"/>
         <geometry>
-          <box size="1.0 0.60 0.60"/>
+          <box size="1.30 0.90 0.90"/>
         </geometry>
         <material name="LightGrey">
@@ -32,6 +33,6 @@
     <parent link="robot_base" />
     <child link = "arm_base_link" />
-    <origin xyz="0.324 -0.191 0.2925" rpy="0.0 0.0 -2.3562" />
-  </joint>
+    <origin xyz="0.0 0.0 0.45" rpy="0.0 0.0 -2.3562" />
+  </joint-->
   <!-- arm -->
   <xacro:ur10_robot prefix="arm_" joint_limited="false"/>

Commit message: remove base

File: ur_description/urdf/ur10_joint_limited_robot.urdf.xacro (robot description, xacro)
@@ -6,32 +6,34 @@
   <!-- ur10 -->
   <xacro:include filename="$(find ur_description)/urdf/ur10.urdf.xacro" />
-  <!--link name="world" />
+  <link name="world" />
   <joint name="world_joint" type="fixed">
     <parent link="world" />
     <child link = "base_link" />
     <origin xyz="0.0 0.0 0.0" rpy="0.0 0.0 0.0" />
-  </joint-->
-    <link name="world" />
-    <joint name="world-robot_base_joint" type="fixed">
-        <origin xyz="-0.65 -0.45 0.45" rpy="0 0 0" />
-        <parent link="world"/>
-        <child link="robot_base"/>
-    </joint>
-    <link name="robot_base">
-        <visual>
-            <origin rpy="0 0 0" xyz="0 0 0"/>
-            <geometry>
-                <box size="1.30 0.90 0.90"/>
-            </geometry>
-            <material name="LightGrey">
-                <color rgba="0.7 0.7 0.7 1.0"/>
-            </material>
-        </visual>
-    </link>
-    <joint name="world_joint" type="fixed">
-        <parent link="robot_base" />
-        <child link = "arm_base_link" />
-        <origin xyz="0.324 -0.191 0.2925" rpy="0.0 0.0 -2.3562" />
-    </joint>
+  </joint>
+  <!--
+ <link name="world" />
+ <joint name="world-robot_base_joint" type="fixed">
+   <origin xyz="-0.50 -0.30 0.30" rpy="0 0 0" />
+   <parent link="world"/>
+   <child link="robot_base"/>
+ </joint>
+ <link name="robot_base">
+     <visual>
+       <origin rpy="0 0 0" xyz="0 0 0"/>
+       <geometry>
+         <box size="1.0 0.60 0.60"/>
+       </geometry>
+       <material name="LightGrey">
+         <color rgba="0.7 0.7 0.7 1.0"/>
+       </material>
+     </visual>
+ </link>
+ <joint name="world_joint" type="fixed">
+   <parent link="robot_base" />
+   <child link = "arm_base_link" />
+   <origin xyz="0.324 -0.191 0.2925" rpy="0.0 0.0 -2.3562" />
+ </joint>
+  -->
     <!-- arm -->
     <xacro:ur10_robot prefix="arm_" joint_limited="true"

File: ur_description/urdf/ur10_robot.urdf.xacro (robot description, xacro)
@@ -6,10 +6,11 @@
   <!-- ur10 -->
   <xacro:include filename="$(find ur_description)/urdf/ur10.urdf.xacro" />
-  <!--link name="world" />
+  <link name="world" />
   <joint name="world_joint" type="fixed">
     <parent link="world" />
     <child link = "arm_base_link" />
     <origin xyz="0.0 0.0 0.0" rpy="0.0 0.0 0.0" />
-  </joint-->
+  </joint>
+ <!--
  <link name="world" />
   <joint name="world-robot_base_joint" type="fixed">
@@ -34,4 +35,5 @@
     <origin xyz="0.324 -0.191 0.2925" rpy="0.0 0.0 -2.3562" />
   </joint>
+  -->
   <!-- arm -->
   <xacro:ur10_robot prefix="arm_" joint_limited="false"/>

Commit message: undo joint limits to standard one

File: ur_description/urdf/ur10_joint_limited_robot.urdf.xacro (robot description, xacro)
@@ -14,10 +14,10 @@
   <!-- arm -->
   <xacro:ur10_robot prefix="" joint_limited="true"
-               shoulder_pan_lower_limit="${-pi}" shoulder_pan_upper_limit="${2.75}"
-               shoulder_lift_lower_limit="${-pi}" shoulder_lift_upper_limit="${pi}"
-               elbow_joint_lower_limit="${-pi}" elbow_joint_upper_limit="${0.2}"
-               wrist_1_lower_limit="${-2*pi}" wrist_1_upper_limit="${-0.5}"
+               shoulder_pan_lower_limit="${-pi}" shoulder_pan_upper_limit="${pi}"
+    	       shoulder_lift_lower_limit="${-pi}" shoulder_lift_upper_limit="${pi}"
+               elbow_joint_lower_limit="${-pi}" elbow_joint_upper_limit="${pi}"
+               wrist_1_lower_limit="${-pi}" wrist_1_upper_limit="${pi}"
                wrist_2_lower_limit="${-pi}" wrist_2_upper_limit="${pi}"
-               wrist_3_lower_limit="${0.5-pi}" wrist_3_upper_limit="${0.5*pi}"
+               wrist_3_lower_limit="${-pi}" wrist_3_upper_limit="${pi}"
   />
   <!-- ros_control plugin -->

File: ur_description/urdf/ur10_robot.urdf.xacro (robot description, xacro)
@@ -12,27 +12,4 @@
     <origin xyz="0.0 0.0 0.0" rpy="0.0 0.0 0.0" />
   </joint>
- <!-- inlcuding table top robot arm -->
- <!--link name="world" />
-  <joint name="world-robot_base_joint" type="fixed">
-    <origin xyz="-0.65 -0.45 0.45" rpy="0 0 0" />
-    <parent link="world"/>
-    <child link="robot_base"/>
-  </joint>
-  <link name="robot_base">
-      <visual>
-        <origin rpy="0 0 0" xyz="0 0 0"/>
-        <geometry>
-          <box size="1.30 0.90 0.90"/>
-        </geometry>
-        <material name="LightGrey">
-          <color rgba="0.7 0.7 0.7 1.0"/>
-        </material>
-      </visual>
-  </link>
-  <joint name="world_joint" type="fixed">
-    <parent link="robot_base" />
-    <child link = "base_link" />
-    <origin xyz="0.0 0.0 0.45" rpy="0.0 0.0 -2.3562" />
-  </joint-->
   <!-- arm -->
   <xacro:ur10_robot prefix="" joint_limited="false"/>
