Commit message: add dummy robot base

File: ur_description/urdf/ur10_robot.urdf.xacro (robot description, xacro)
@@ -12,8 +12,24 @@
   />
   <link name="world" />
+  <joint name="world-robot_base_joint" type="fixed">
+    <origin xyz="-0.50 -0.30 0.30" rpy="0 0 0" />
+    <parent link="world"/>
+    <child link="robot_base"/>
+  </joint>
+  <link name="robot_base">
+      <visual>
+        <origin rpy="0 0 0" xyz="0 0 0"/>
+        <geometry>
+          <box size="1.0 0.60 0.60"/>
+        </geometry>
+        <material name="LightGrey">
+          <color rgba="0.7 0.7 0.7 1.0"/>
+        </material>
+      </visual>
+  </link>
   <joint name="world_joint" type="fixed">
-    <parent link="world" />
+    <parent link="robot_base" />
     <child link = "base_link" />
-    <origin xyz="0.0 0.0 0.0" rpy="0.0 0.0 0.0" />
+    <origin xyz="0.324 -0.191 0.2925" rpy="0.0 0.0 -2.3562" />
   </joint>
 </robot>

Commit message: added velocity control to ur10

File: ur_description/urdf/ur10_robot.urdf.xacro (robot description, xacro)
@@ -6,11 +6,18 @@
   <!-- ur10 -->
   <xacro:include filename="$(find ur_description)/urdf/ur10.urdf.xacro" />
-  <!-- arm -->
-  <xacro:ur10_robot prefix="" joint_limited="false"/>
   <link name="world" />
   <joint name="world_joint" type="fixed">
     <parent link="world" />
-    <child link = "base_link" />
+    <child link = "arm_base_link" />
     <origin xyz="0.0 0.0 0.0" rpy="0.0 0.0 0.0" />
   </joint>
+  <!-- arm -->
+  <xacro:ur10_robot prefix="arm_" joint_limited="false"/>
+  <!-- ros_control plugin -->
+  <gazebo>
+    <plugin name="ros_control" filename="libhwi_switch_gazebo_ros_control.so">
+      <robotNamespace>arm</robotNamespace>
+      <filterJointsParam>joint_names</filterJointsParam>
+    </plugin>
+  </gazebo>
 </robot>

Commit message: add dummy base as box

File: ur_description/urdf/ur10_robot.urdf.xacro (robot description, xacro)
@@ -6,9 +6,31 @@
   <!-- ur10 -->
   <xacro:include filename="$(find ur_description)/urdf/ur10.urdf.xacro" />
-  <link name="world" />
+  <!--link name="world" />
   <joint name="world_joint" type="fixed">
     <parent link="world" />
     <child link = "arm_base_link" />
     <origin xyz="0.0 0.0 0.0" rpy="0.0 0.0 0.0" />
+  </joint-->
+ <link name="world" />
+  <joint name="world-robot_base_joint" type="fixed">
+    <origin xyz="-0.50 -0.30 0.30" rpy="0 0 0" />
+    <parent link="world"/>
+    <child link="robot_base"/>
+  </joint>
+  <link name="robot_base">
+      <visual>
+        <origin rpy="0 0 0" xyz="0 0 0"/>
+        <geometry>
+          <box size="1.0 0.60 0.60"/>
+        </geometry>
+        <material name="LightGrey">
+          <color rgba="0.7 0.7 0.7 1.0"/>
+        </material>
+      </visual>
+  </link>
+  <joint name="world_joint" type="fixed">
+    <parent link="robot_base" />
+    <child link = "arm_base_link" />
+    <origin xyz="0.324 -0.191 0.2925" rpy="0.0 0.0 -2.3562" />
   </joint>
   <!-- arm -->

Commit message: comment table

File: ur_description/urdf/ur10_robot.urdf.xacro (robot description, xacro)
@@ -6,14 +6,12 @@
   <!-- ur10 -->
   <xacro:include filename="$(find ur_description)/urdf/ur10.urdf.xacro" />
-  <!--
   <link name="world" />
   <joint name="world_joint" type="fixed">
     <parent link="world" />
-    <child link = "arm_base_link" />
+    <child link = "base_link" />
     <origin xyz="0.0 0.0 0.0" rpy="0.0 0.0 0.0" />
   </joint>
-  -->
  <!-- inlcuding table top robot arm -->
- <link name="world" />
+ <!--link name="world" />
   <joint name="world-robot_base_joint" type="fixed">
     <origin xyz="-0.65 -0.45 0.45" rpy="0 0 0" />
@@ -36,5 +34,5 @@
     <child link = "base_link" />
     <origin xyz="0.0 0.0 0.45" rpy="0.0 0.0 -2.3562" />
-  </joint>
+  </joint-->
   <!-- arm -->
   <xacro:ur10_robot prefix="" joint_limited="false"/>

Commit message: added robotiq gripper in urdf model, still not perfect

File: ur_description/urdf/ur10_robot.urdf.xacro (robot description, xacro)
@@ -6,4 +6,6 @@
   <!-- ur10 -->
   <xacro:include filename="$(find ur_description)/urdf/ur10.urdf.xacro" />
+  <!-- Robotiq Gripper attached -->
+  <xacro:include filename="$(find robotiq_85_description)/urdf/robotiq_85_gripper.urdf.xacro" />
   <link name="world" />
   <joint name="world_joint" type="fixed">
@@ -14,4 +16,8 @@
   <!-- arm -->
   <xacro:ur10_robot prefix="" joint_limited="false"/>
+  <!-- gripper-->
+  <xacro:robotiq_85_gripper prefix="" parent="wrist_3_link">
+    <origin xyz="0.0 0.09 0.0" rpy="0.0 0.0 ${3.1415/2.0}" />
+  </xacro:robotiq_85_gripper>
   <!-- ros_control plugin -->
   <gazebo>
