Commit message: changed name of joint to avoid diferent alphabatic order

File: ur_description/urdf/ur10.urdf.xacro (robot description, xacro)
@@ -54,7 +54,7 @@
   </xacro:macro>
   <xacro:macro name="ur10_robot" params="prefix joint_limited
-		 shoulder_pan_lower_limit:=${-0.5*pi}    shoulder_pan_upper_limit:=${0.2}
+		 shoulder_pan_lower_limit:=${-0.5*pi}    shoulder_pan_upper_limit:=${0.5}
 		 shoulder_lift_lower_limit:=${-pi}    shoulder_lift_upper_limit:=${pi}
-		 elbow_joint_lower_limit:=${-pi}    elbow_joint_upper_limit:=${0.2}
+		 shoulder_3_joint_lower_limit:=${-pi}    shoulder_3_joint_upper_limit:=${0.2}
 		 wrist_1_lower_limit:=${-2*pi}    wrist_1_upper_limit:=${-0.5}
 		 wrist_2_lower_limit:=${-pi}    wrist_2_upper_limit:=${pi}
@@ -78,5 +78,5 @@
       </xacro:cylinder_inertial>
     </link>
-    <joint name="${prefix}shoulder_pan_joint" type="revolute">
+    <joint name="${prefix}shoulder_1_joint" type="revolute">
       <parent link="${prefix}base_link" />
       <child link = "${prefix}shoulder_link" />
@@ -109,5 +109,5 @@
       </xacro:cylinder_inertial>
     </link>
-    <joint name="${prefix}shoulder_lift_joint" type="revolute">
+    <joint name="${prefix}shoulder_2_joint" type="revolute">
       <parent link="${prefix}shoulder_link" />
       <child link = "${prefix}upper_arm_link" />
@@ -140,5 +140,5 @@
       </xacro:cylinder_inertial>
     </link>
-    <joint name="${prefix}elbow_joint" type="revolute">
+    <joint name="${prefix}shoulder_3_joint" type="revolute">
       <parent link="${prefix}upper_arm_link" />
       <child link = "${prefix}forearm_link" />
@@ -149,5 +149,5 @@
       </xacro:unless>
       <xacro:if value="${joint_limited}">
-        <limit lower="${elbow_joint_lower_limit}" upper="${elbow_joint_upper_limit}" effort="150.0" velocity="3.15"/>
+        <limit lower="${shoulder_3_joint_lower_limit}" upper="${shoulder_3_joint_upper_limit}" effort="150.0" velocity="3.15"/>
       </xacro:if>
       <dynamics damping="0.0" friction="0.0"/>

File: ur_description/urdf/ur10_joint_limited_robot.urdf.xacro (robot description, xacro)
@@ -8,7 +8,7 @@
   <!-- arm -->
   <xacro:ur10_robot prefix="" joint_limited="true"
-		 shoulder_pan_lower_limit="${-pi}" shoulder_pan_upper_limit="${pi}"
-		 shoulder_lift_lower_limit="${-pi}" shoulder_lift_upper_limit="${pi}"
-		 elbow_joint_lower_limit="${-pi}" elbow_joint_upper_limit="${pi}"
+		 shoulder_1_lower_limit="${-pi}" shoulder_1_upper_limit="${pi}"
+		 shoulder_2_lower_limit="${-pi}" shoulder_2_upper_limit="${pi}"
+		 shoulder_3_joint_lower_limit="${-pi}" shoulder_3_joint_upper_limit="${pi}"
 		 wrist_1_lower_limit="${-pi}" wrist_1_upper_limit="${pi}"
 		 wrist_2_lower_limit="${-pi}" wrist_2_upper_limit="${pi}"

Commit message: joint speed limits changed

File: ur_description/urdf/ur10.urdf.xacro (robot description, xacro)
@@ -84,8 +84,8 @@
       <axis xyz="0 0 1" />
       <xacro:unless value="${joint_limited}">
-        <limit lower="${-2.0 * pi}" upper="${2.0 * pi}" effort="330.0" velocity="2.16"/>
-      </xacro:unless>
-      <xacro:if value="${joint_limited}">
-        <limit lower="${shoulder_pan_lower_limit}" upper="${shoulder_pan_upper_limit}" effort="330.0" velocity="2.16"/>
+        <limit lower="${-2.0 * pi}" upper="${2.0 * pi}" effort="330.0" velocity="2.0"/>
+      </xacro:unless>
+      <xacro:if value="${joint_limited}">
+        <limit lower="${shoulder_pan_lower_limit}" upper="${shoulder_pan_upper_limit}" effort="330.0" velocity="2.0"/>
       </xacro:if>
       <dynamics damping="0.0" friction="0.0"/>
@@ -115,8 +115,8 @@
       <axis xyz="0 1 0" />
       <xacro:unless value="${joint_limited}">
-        <limit lower="${-2.0 * pi}" upper="${2.0 * pi}" effort="330.0" velocity="2.16"/>
-      </xacro:unless>
-      <xacro:if value="${joint_limited}">
-        <limit lower="${shoulder_lift_lower_limit}" upper="${shoulder_lift_upper_limit}" effort="330.0" velocity="2.16"/>
+        <limit lower="${-2.0 * pi}" upper="${2.0 * pi}" effort="330.0" velocity="2.0"/>
+      </xacro:unless>
+      <xacro:if value="${joint_limited}">
+        <limit lower="${shoulder_lift_lower_limit}" upper="${shoulder_lift_upper_limit}" effort="330.0" velocity="2.0"/>
       </xacro:if>
       <dynamics damping="0.0" friction="0.0"/>
@@ -146,8 +146,8 @@
       <axis xyz="0 1 0" />
       <xacro:unless value="${joint_limited}">
-        <limit lower="${-pi}" upper="${pi}" effort="150.0" velocity="3.15"/>
-      </xacro:unless>
-      <xacro:if value="${joint_limited}">
-        <limit lower="${elbow_joint_lower_limit}" upper="${elbow_joint_upper_limit}" effort="150.0" velocity="3.15"/>
+        <limit lower="${-2.0 * pi}" upper="${2.0 * pi}" effort="150.0" velocity="2.0"/>
+      </xacro:unless>
+      <xacro:if value="${joint_limited}">
+        <limit lower="${elbow_joint_lower_limit}" upper="${elbow_joint_upper_limit}" effort="150.0" velocity="2.0"/>
       </xacro:if>
       <dynamics damping="0.0" friction="0.0"/>
@@ -177,8 +177,8 @@
       <axis xyz="0 1 0" />
       <xacro:unless value="${joint_limited}">
-        <limit lower="${-2.0 * pi}" upper="${2.0 * pi}" effort="54.0" velocity="3.2"/>
-      </xacro:unless>
-      <xacro:if value="${joint_limited}">
-        <limit lower="${wrist_1_lower_limit}" upper="${wrist_1_upper_limit}" effort="54.0" velocity="3.2"/>
+        <limit lower="${-2.0 * pi}" upper="${2.0 * pi}" effort="54.0" velocity="2.0"/>
+      </xacro:unless>
+      <xacro:if value="${joint_limited}">
+        <limit lower="${wrist_1_lower_limit}" upper="${wrist_1_upper_limit}" effort="54.0" velocity="2.0"/>
       </xacro:if>
       <dynamics damping="0.0" friction="0.0"/>
@@ -208,8 +208,8 @@
       <axis xyz="0 0 1" />
       <xacro:unless value="${joint_limited}">
-        <limit lower="${-2.0 * pi}" upper="${2.0 * pi}" effort="54.0" velocity="3.2"/>
-      </xacro:unless>
-      <xacro:if value="${joint_limited}">
-        <limit lower="${wrist_2_lower_limit}" upper="${wrist_2_upper_limit}" effort="54.0" velocity="3.2"/>
+        <limit lower="${-2.0 * pi}" upper="${2.0 * pi}" effort="54.0" velocity="2.0"/>
+      </xacro:unless>
+      <xacro:if value="${joint_limited}">
+        <limit lower="${wrist_2_lower_limit}" upper="${wrist_2_upper_limit}" effort="54.0" velocity="2.0"/>
       </xacro:if>
       <dynamics damping="0.0" friction="0.0"/>
@@ -239,8 +239,8 @@
       <axis xyz="0 1 0" />
       <xacro:unless value="${joint_limited}">
-        <limit lower="${-2.0 * pi}" upper="${2.0 * pi}" effort="54.0" velocity="3.2"/>
-      </xacro:unless>
-      <xacro:if value="${joint_limited}">
-        <limit lower="${wrist_3_lower_limit}" upper="${wrist_3_upper_limit}" effort="54.0" velocity="3.2"/>
+        <limit lower="${-2.0 * pi}" upper="${2.0 * pi}" effort="54.0" velocity="2.0"/>
+      </xacro:unless>
+      <xacro:if value="${joint_limited}">
+        <limit lower="${wrist_3_lower_limit}" upper="${wrist_3_upper_limit}" effort="54.0" velocity="2.0"/>
       </xacro:if>
       <dynamics damping="0.0" friction="0.0"/>

Commit message: joint speed limits changed

File: ur_description/urdf/ur10.urdf.xacro (robot description, xacro)
@@ -84,8 +84,8 @@
       <axis xyz="0 0 1" />
       <xacro:unless value="${joint_limited}">
-        <limit lower="${-2.0 * pi}" upper="${2.0 * pi}" effort="330.0" velocity="2.16"/>
-      </xacro:unless>
-      <xacro:if value="${joint_limited}">
-        <limit lower="${shoulder_pan_lower_limit}" upper="${shoulder_pan_upper_limit}" effort="330.0" velocity="2.16"/>
+        <limit lower="${-2.0 * pi}" upper="${2.0 * pi}" effort="330.0" velocity="2.0"/>
+      </xacro:unless>
+      <xacro:if value="${joint_limited}">
+        <limit lower="${shoulder_pan_lower_limit}" upper="${shoulder_pan_upper_limit}" effort="330.0" velocity="2.0"/>
       </xacro:if>
       <dynamics damping="0.0" friction="0.0"/>
@@ -115,8 +115,8 @@
       <axis xyz="0 1 0" />
       <xacro:unless value="${joint_limited}">
-        <limit lower="${-2.0 * pi}" upper="${2.0 * pi}" effort="330.0" velocity="2.16"/>
-      </xacro:unless>
-      <xacro:if value="${joint_limited}">
-        <limit lower="${shoulder_lift_lower_limit}" upper="${shoulder_lift_upper_limit}" effort="330.0" velocity="2.16"/>
+        <limit lower="${-2.0 * pi}" upper="${2.0 * pi}" effort="330.0" velocity="2.0"/>
+      </xacro:unless>
+      <xacro:if value="${joint_limited}">
+        <limit lower="${shoulder_lift_lower_limit}" upper="${shoulder_lift_upper_limit}" effort="330.0" velocity="2.0"/>
       </xacro:if>
       <dynamics damping="0.0" friction="0.0"/>
@@ -146,8 +146,8 @@
       <axis xyz="0 1 0" />
       <xacro:unless value="${joint_limited}">
-        <limit lower="${-2.0 * pi}" upper="${2.0 * pi}" effort="150.0" velocity="3.15"/>
-      </xacro:unless>
-      <xacro:if value="${joint_limited}">
-        <limit lower="${elbow_joint_lower_limit}" upper="${elbow_joint_upper_limit}" effort="150.0" velocity="3.15"/>
+        <limit lower="${-2.0 * pi}" upper="${2.0 * pi}" effort="150.0" velocity="2.0"/>
+      </xacro:unless>
+      <xacro:if value="${joint_limited}">
+        <limit lower="${elbow_joint_lower_limit}" upper="${elbow_joint_upper_limit}" effort="150.0" velocity="2.0"/>
       </xacro:if>
       <dynamics damping="0.0" friction="0.0"/>
@@ -177,8 +177,8 @@
       <axis xyz="0 1 0" />
       <xacro:unless value="${joint_limited}">
-        <limit lower="${-2.0 * pi}" upper="${2.0 * pi}" effort="54.0" velocity="3.2"/>
-      </xacro:unless>
-      <xacro:if value="${joint_limited}">
-        <limit lower="${wrist_1_lower_limit}" upper="${wrist_1_upper_limit}" effort="54.0" velocity="3.2"/>
+        <limit lower="${-2.0 * pi}" upper="${2.0 * pi}" effort="54.0" velocity="2.0"/>
+      </xacro:unless>
+      <xacro:if value="${joint_limited}">
+        <limit lower="${wrist_1_lower_limit}" upper="${wrist_1_upper_limit}" effort="54.0" velocity="2.0"/>
       </xacro:if>
       <dynamics damping="0.0" friction="0.0"/>
@@ -208,8 +208,8 @@
       <axis xyz="0 0 1" />
       <xacro:unless value="${joint_limited}">
-        <limit lower="${-2.0 * pi}" upper="${2.0 * pi}" effort="54.0" velocity="3.2"/>
-      </xacro:unless>
-      <xacro:if value="${joint_limited}">
-        <limit lower="${wrist_2_lower_limit}" upper="${wrist_2_upper_limit}" effort="54.0" velocity="3.2"/>
+        <limit lower="${-2.0 * pi}" upper="${2.0 * pi}" effort="54.0" velocity="2.0"/>
+      </xacro:unless>
+      <xacro:if value="${joint_limited}">
+        <limit lower="${wrist_2_lower_limit}" upper="${wrist_2_upper_limit}" effort="54.0" velocity="2.0"/>
       </xacro:if>
       <dynamics damping="0.0" friction="0.0"/>
@@ -239,8 +239,8 @@
       <axis xyz="0 1 0" />
       <xacro:unless value="${joint_limited}">
-        <limit lower="${-2.0 * pi}" upper="${2.0 * pi}" effort="54.0" velocity="3.2"/>
-      </xacro:unless>
-      <xacro:if value="${joint_limited}">
-        <limit lower="${wrist_3_lower_limit}" upper="${wrist_3_upper_limit}" effort="54.0" velocity="3.2"/>
+        <limit lower="${-2.0 * pi}" upper="${2.0 * pi}" effort="54.0" velocity="2.0"/>
+      </xacro:unless>
+      <xacro:if value="${joint_limited}">
+        <limit lower="${wrist_3_lower_limit}" upper="${wrist_3_upper_limit}" effort="54.0" velocity="2.0"/>
       </xacro:if>
       <dynamics damping="0.0" friction="0.0"/>

Commit message: tool0 frame joint and link changed for bumper sensor

File: ur_description/urdf/ur10.urdf.xacro (robot description, xacro)
@@ -291,9 +291,23 @@
     </joint>
     <!-- Frame coincident with all-zeros TCP on UR controller -->
-    <link name="${prefix}tool0"/>
+    <link name="${prefix}tool0">
+      <collision>
+        <geometry>
+          <box size="0.01 0.01 0.01"/>
+        </geometry>
+        <origin rpy="0 0 0" xyz="-0.01 0 0"/>
+      </collision>
+    </link>
     <joint name="${prefix}wrist_3_link-tool0_fixed_joint" type="fixed">
-      <origin xyz="0 ${wrist_3_length} 0" rpy="${pi/-2.0} 0 0"/>
+      <origin xyz="0.0 0.2922 0.0" rpy="0.0 0.0 ${pi/2.0}" />
       <parent link="${prefix}wrist_3_link"/>
       <child link="${prefix}tool0"/>
+      <xacro:unless value="${joint_limited}">
+        <limit lower="${-2.0 * pi}" upper="${2.0 * pi}" effort="54.0" velocity="3.2"/>
+      </xacro:unless>
+      <xacro:if value="${joint_limited}">
+        <limit lower="${wrist_3_lower_limit}" upper="${wrist_3_upper_limit}" effort="54.0" velocity="3.2"/>
+      </xacro:if>
+      <dynamics damping="0.0" friction="0.0"/>
     </joint>
   </xacro:macro>

Commit message: change joint name from urdf

File: ur_description/urdf/ur10.urdf.xacro (robot description, xacro)
@@ -54,7 +54,7 @@
   </xacro:macro>
   <xacro:macro name="ur10_robot" params="prefix joint_limited
-		 shoulder_1_joint_lower_limit:=${-pi}    shoulder_1_joint_upper_limit:=${0.5}
-		 shoulder_2_joint_lower_limit:=${-pi}    shoulder_2_joint_upper_limit:=${pi}
-		 shoulder_3_joint_lower_limit:=${-pi}    shoulder_3_joint_upper_limit:=${0.2}
+		 shoulder_pan_lower_limit:=${-pi}    shoulder_pan_upper_limit:=${0.2}
+		 shoulder_lift_lower_limit:=${-pi}    shoulder_lift_upper_limit:=${pi}
+		 elbow_joint_lower_limit:=${-pi}    elbow_joint_upper_limit:=${0.2}
 		 wrist_1_lower_limit:=${-2*pi}    wrist_1_upper_limit:=${-0.5}
 		 wrist_2_lower_limit:=${-pi}    wrist_2_upper_limit:=${pi}
@@ -78,5 +78,5 @@
       </xacro:cylinder_inertial>
     </link>
-    <joint name="${prefix}shoulder_1_joint" type="revolute">
+    <joint name="${prefix}shoulder_pan_joint" type="revolute">
       <parent link="${prefix}base_link" />
       <child link = "${prefix}shoulder_link" />
@@ -84,8 +84,8 @@
       <axis xyz="0 0 1" />
       <xacro:unless value="${joint_limited}">
-        <limit lower="${-2.0 * pi}" upper="${2.0 * pi}" effort="330.0" velocity="2.16"/>
-      </xacro:unless>
-      <xacro:if value="${joint_limited}">
-        <limit lower="${shoulder_1_joint_lower_limit}" upper="${shoulder_1_joint_upper_limit}" effort="330.0" velocity="2.16"/>
+        <limit lower="${-2.0 * pi}" upper="${2.0 * pi}" effort="330.0" velocity="2.0"/>
+      </xacro:unless>
+      <xacro:if value="${joint_limited}">
+        <limit lower="${shoulder_pan_lower_limit}" upper="${shoulder_pan_upper_limit}" effort="330.0" velocity="2.0"/>
       </xacro:if>
       <dynamics damping="0.0" friction="0.0"/>
@@ -109,5 +109,5 @@
       </xacro:cylinder_inertial>
     </link>
-    <joint name="${prefix}shoulder_2_joint" type="revolute">
+    <joint name="${prefix}shoulder_lift_joint" type="revolute">
       <parent link="${prefix}shoulder_link" />
       <child link = "${prefix}upper_arm_link" />
@@ -115,8 +115,8 @@
       <axis xyz="0 1 0" />
       <xacro:unless value="${joint_limited}">
-        <limit lower="${-2.0 * pi}" upper="${2.0 * pi}" effort="330.0" velocity="2.16"/>
-      </xacro:unless>
-      <xacro:if value="${joint_limited}">
-        <limit lower="${shoulder_2_joint_lower_limit}" upper="${shoulder_2_joint_upper_limit}" effort="330.0" velocity="2.16"/>
+        <limit lower="${-2.0 * pi}" upper="${2.0 * pi}" effort="330.0" velocity="2.0"/>
+      </xacro:unless>
+      <xacro:if value="${joint_limited}">
+        <limit lower="${shoulder_lift_lower_limit}" upper="${shoulder_lift_upper_limit}" effort="330.0" velocity="2.0"/>
       </xacro:if>
       <dynamics damping="0.0" friction="0.0"/>
@@ -140,5 +140,5 @@
       </xacro:cylinder_inertial>
     </link>
-    <joint name="${prefix}shoulder_3_joint" type="revolute">
+    <joint name="${prefix}elbow_joint" type="revolute">
       <parent link="${prefix}upper_arm_link" />
       <child link = "${prefix}forearm_link" />
@@ -146,8 +146,8 @@
       <axis xyz="0 1 0" />
       <xacro:unless value="${joint_limited}">
-        <limit lower="${-2.0 * pi}" upper="${2.0 * pi}" effort="150.0" velocity="3.15"/>
-      </xacro:unless>
-      <xacro:if value="${joint_limited}">
-        <limit lower="${shoulder_3_joint_lower_limit}" upper="${shoulder_3_joint_upper_limit}" effort="150.0" velocity="3.15"/>
+        <limit lower="${-2.0 * pi}" upper="${2.0 * pi}" effort="150.0" velocity="2.0"/>
+      </xacro:unless>
+      <xacro:if value="${joint_limited}">
+        <limit lower="${elbow_joint_lower_limit}" upper="${elbow_joint_upper_limit}" effort="150.0" velocity="2.0"/>
       </xacro:if>
       <dynamics damping="0.0" friction="0.0"/>
@@ -177,8 +177,8 @@
       <axis xyz="0 1 0" />
       <xacro:unless value="${joint_limited}">
-        <limit lower="${-2.0 * pi}" upper="${2.0 * pi}" effort="54.0" velocity="3.2"/>
-      </xacro:unless>
-      <xacro:if value="${joint_limited}">
-        <limit lower="${wrist_1_lower_limit}" upper="${wrist_1_upper_limit}" effort="54.0" velocity="3.2"/>
+        <limit lower="${-2.0 * pi}" upper="${2.0 * pi}" effort="54.0" velocity="2.0"/>
+      </xacro:unless>
+      <xacro:if value="${joint_limited}">
+        <limit lower="${wrist_1_lower_limit}" upper="${wrist_1_upper_limit}" effort="54.0" velocity="2.0"/>
       </xacro:if>
       <dynamics damping="0.0" friction="0.0"/>
@@ -208,8 +208,8 @@
       <axis xyz="0 0 1" />
       <xacro:unless value="${joint_limited}">
-        <limit lower="${-2.0 * pi}" upper="${2.0 * pi}" effort="54.0" velocity="3.2"/>
-      </xacro:unless>
-      <xacro:if value="${joint_limited}">
-        <limit lower="${wrist_2_lower_limit}" upper="${wrist_2_upper_limit}" effort="54.0" velocity="3.2"/>
+        <limit lower="${-2.0 * pi}" upper="${2.0 * pi}" effort="54.0" velocity="2.0"/>
+      </xacro:unless>
+      <xacro:if value="${joint_limited}">
+        <limit lower="${wrist_2_lower_limit}" upper="${wrist_2_upper_limit}" effort="54.0" velocity="2.0"/>
       </xacro:if>
       <dynamics damping="0.0" friction="0.0"/>
@@ -239,8 +239,8 @@
       <axis xyz="0 1 0" />
       <xacro:unless value="${joint_limited}">
-        <limit lower="${-2.0 * pi}" upper="${2.0 * pi}" effort="54.0" velocity="3.2"/>
-      </xacro:unless>
-      <xacro:if value="${joint_limited}">
-        <limit lower="${wrist_3_lower_limit}" upper="${wrist_3_upper_limit}" effort="54.0" velocity="3.2"/>
+        <limit lower="${-2.0 * pi}" upper="${2.0 * pi}" effort="54.0" velocity="2.0"/>
+      </xacro:unless>
+      <xacro:if value="${joint_limited}">
+        <limit lower="${wrist_3_lower_limit}" upper="${wrist_3_upper_limit}" effort="54.0" velocity="2.0"/>
       </xacro:if>
       <dynamics damping="0.0" friction="0.0"/>

Commit message: change joint mass value make it same as indigo_dev

File: ur_description/urdf/ur10.urdf.xacro (robot description, xacro)
@@ -10,10 +10,10 @@
   <!-- Inertia parameters -->
   <xacro:property name="base_mass" value="4.0" />  <!-- This mass might be incorrect -->
-  <xacro:property name="shoulder_mass" value="7.778" />
-  <xacro:property name="upper_arm_mass" value="12.93" />
-  <xacro:property name="forearm_mass" value="3.87" />
-  <xacro:property name="wrist_1_mass" value="1.96" />
-  <xacro:property name="wrist_2_mass" value="1.96" />
-  <xacro:property name="wrist_3_mass" value="0.202" />
+  <xacro:property name="shoulder_mass" value="1" />
+  <xacro:property name="upper_arm_mass" value="1" />
+  <xacro:property name="forearm_mass" value="1" />
+  <xacro:property name="wrist_1_mass" value="0.5" />
+  <xacro:property name="wrist_2_mass" value="0.5" />
+  <xacro:property name="wrist_3_mass" value="0.5" />
   <!-- These parameters are borrowed from the urcontrol.conf file
        but are not verified for the correct permutation.
@@ -300,5 +300,5 @@
     </link>
     <joint name="${prefix}wrist_3_link-tool0_fixed_joint" type="fixed">
-      <origin xyz="0.0 0.2922 0.0" rpy="0.0 0.0 ${pi/2.0}" />
+      <origin xyz="0.0 ${wrist_3_length+0.14} 0.0" rpy="0.0 0.0 ${pi/2.0}" />
       <parent link="${prefix}wrist_3_link"/>
       <child link="${prefix}tool0"/>
