Commit message: merge with stomp

File: ur_description/urdf/ur10.urdf.xacro (robot description, xacro)
@@ -7,4 +7,5 @@
   <xacro:include filename="$(find ur_description)/urdf/ur.transmission.xacro" />
   <xacro:include filename="$(find ur_description)/urdf/ur.gazebo.xacro" />
+  <xacro:property name="pi" value="3.14159265" />
   <!-- Inertia parameters -->
   <xacro:property name="base_mass" value="4.0" />  <!-- This mass might be incorrect -->
@@ -53,10 +54,10 @@
   </xacro:macro>
   <xacro:macro name="ur10_robot" params="prefix joint_limited
-		 shoulder_pan_lower_limit:=${-pi}    shoulder_pan_upper_limit:=${pi}
+		 shoulder_pan_lower_limit:=${-0.5*pi}    shoulder_pan_upper_limit:=${0.2}
 		 shoulder_lift_lower_limit:=${-pi}    shoulder_lift_upper_limit:=${pi}
-		 elbow_joint_lower_limit:=${-pi}    elbow_joint_upper_limit:=${pi}
-		 wrist_1_lower_limit:=${-pi}    wrist_1_upper_limit:=${pi}
+		 elbow_joint_lower_limit:=${-pi}    elbow_joint_upper_limit:=${0.2}
+		 wrist_1_lower_limit:=${-2*pi}    wrist_1_upper_limit:=${-0.5}
 		 wrist_2_lower_limit:=${-pi}    wrist_2_upper_limit:=${pi}
-		 wrist_3_lower_limit:=${-pi}    wrist_3_upper_limit:=${pi}">
+		 wrist_3_lower_limit:=${0.5-pi}    wrist_3_upper_limit:=${0.5*pi}">
     <link name="${prefix}base_link" >
       <visual>
@@ -83,8 +84,8 @@
       <axis xyz="0 0 1" />
       <xacro:unless value="${joint_limited}">
-        <limit lower="${-2.0 * pi}" upper="${2.0 * pi}" effort="330.0" velocity="2.16"/>
-      </xacro:unless>
-      <xacro:if value="${joint_limited}">
-        <limit lower="${shoulder_pan_lower_limit}" upper="${shoulder_pan_upper_limit}" effort="330.0" velocity="2.16"/>
+        <limit lower="${-2.0 * pi}" upper="${2.0 * pi}" effort="330.0" velocity="2.0"/>
+      </xacro:unless>
+      <xacro:if value="${joint_limited}">
+        <limit lower="${shoulder_pan_lower_limit}" upper="${shoulder_pan_upper_limit}" effort="330.0" velocity="2.0"/>
       </xacro:if>
       <dynamics damping="0.0" friction="0.0"/>
@@ -114,8 +115,8 @@
       <axis xyz="0 1 0" />
       <xacro:unless value="${joint_limited}">
-        <limit lower="${-2.0 * pi}" upper="${2.0 * pi}" effort="330.0" velocity="2.16"/>
-      </xacro:unless>
-      <xacro:if value="${joint_limited}">
-        <limit lower="${shoulder_lift_lower_limit}" upper="${shoulder_lift_upper_limit}" effort="330.0" velocity="2.16"/>
+        <limit lower="${-2.0 * pi}" upper="${2.0 * pi}" effort="330.0" velocity="2.0"/>
+      </xacro:unless>
+      <xacro:if value="${joint_limited}">
+        <limit lower="${shoulder_lift_lower_limit}" upper="${shoulder_lift_upper_limit}" effort="330.0" velocity="2.0"/>
       </xacro:if>
       <dynamics damping="0.0" friction="0.0"/>
@@ -145,8 +146,8 @@
       <axis xyz="0 1 0" />
       <xacro:unless value="${joint_limited}">
-        <limit lower="${-pi}" upper="${pi}" effort="150.0" velocity="3.15"/>
-      </xacro:unless>
-      <xacro:if value="${joint_limited}">
-        <limit lower="${elbow_joint_lower_limit}" upper="${elbow_joint_upper_limit}" effort="150.0" velocity="3.15"/>
+        <limit lower="${-2.0 * pi}" upper="${2.0 * pi}" effort="150.0" velocity="2.0"/>
+      </xacro:unless>
+      <xacro:if value="${joint_limited}">
+        <limit lower="${elbow_joint_lower_limit}" upper="${elbow_joint_upper_limit}" effort="150.0" velocity="2.0"/>
       </xacro:if>
       <dynamics damping="0.0" friction="0.0"/>
@@ -176,8 +177,8 @@
       <axis xyz="0 1 0" />
       <xacro:unless value="${joint_limited}">
-        <limit lower="${-2.0 * pi}" upper="${2.0 * pi}" effort="54.0" velocity="3.2"/>
-      </xacro:unless>
-      <xacro:if value="${joint_limited}">
-        <limit lower="${wrist_1_lower_limit}" upper="${wrist_1_upper_limit}" effort="54.0" velocity="3.2"/>
+        <limit lower="${-2.0 * pi}" upper="${2.0 * pi}" effort="54.0" velocity="2.0"/>
+      </xacro:unless>
+      <xacro:if value="${joint_limited}">
+        <limit lower="${wrist_1_lower_limit}" upper="${wrist_1_upper_limit}" effort="54.0" velocity="2.0"/>
       </xacro:if>
       <dynamics damping="0.0" friction="0.0"/>
@@ -207,8 +208,8 @@
       <axis xyz="0 0 1" />
       <xacro:unless value="${joint_limited}">
-        <limit lower="${-2.0 * pi}" upper="${2.0 * pi}" effort="54.0" velocity="3.2"/>
-      </xacro:unless>
-      <xacro:if value="${joint_limited}">
-        <limit lower="${wrist_2_lower_limit}" upper="${wrist_2_upper_limit}" effort="54.0" velocity="3.2"/>
+        <limit lower="${-2.0 * pi}" upper="${2.0 * pi}" effort="54.0" velocity="2.0"/>
+      </xacro:unless>
+      <xacro:if value="${joint_limited}">
+        <limit lower="${wrist_2_lower_limit}" upper="${wrist_2_upper_limit}" effort="54.0" velocity="2.0"/>
       </xacro:if>
       <dynamics damping="0.0" friction="0.0"/>
@@ -238,8 +239,8 @@
       <axis xyz="0 1 0" />
       <xacro:unless value="${joint_limited}">
-        <limit lower="${-2.0 * pi}" upper="${2.0 * pi}" effort="54.0" velocity="3.2"/>
-      </xacro:unless>
-      <xacro:if value="${joint_limited}">
-        <limit lower="${wrist_3_lower_limit}" upper="${wrist_3_upper_limit}" effort="54.0" velocity="3.2"/>
+        <limit lower="${-2.0 * pi}" upper="${2.0 * pi}" effort="54.0" velocity="2.0"/>
+      </xacro:unless>
+      <xacro:if value="${joint_limited}">
+        <limit lower="${wrist_3_lower_limit}" upper="${wrist_3_upper_limit}" effort="54.0" velocity="2.0"/>
       </xacro:if>
       <dynamics damping="0.0" friction="0.0"/>

Commit message: change velocity limit

File: ur_description/urdf/ur10.urdf.xacro (robot description, xacro)
@@ -54,10 +54,10 @@
   </xacro:macro>
   <xacro:macro name="ur10_robot" params="prefix joint_limited
-		 shoulder_pan_lower_limit:=${-pi}    shoulder_pan_upper_limit:=${pi}
+		 shoulder_pan_lower_limit:=${-0.5*pi}    shoulder_pan_upper_limit:=${0.2}
 		 shoulder_lift_lower_limit:=${-pi}    shoulder_lift_upper_limit:=${pi}
-		 elbow_joint_lower_limit:=${-pi}    elbow_joint_upper_limit:=${pi}
-		 wrist_1_lower_limit:=${-pi}    wrist_1_upper_limit:=${pi}
+		 elbow_joint_lower_limit:=${-pi}    elbow_joint_upper_limit:=${0.2}
+		 wrist_1_lower_limit:=${-2*pi}    wrist_1_upper_limit:=${-0.5}
 		 wrist_2_lower_limit:=${-pi}    wrist_2_upper_limit:=${pi}
-		 wrist_3_lower_limit:=${-pi}    wrist_3_upper_limit:=${pi}">
+		 wrist_3_lower_limit:=${0.5-pi}    wrist_3_upper_limit:=${0.5*pi}">
     <link name="${prefix}base_link" >
       <visual>
@@ -84,8 +84,8 @@
       <axis xyz="0 0 1" />
       <xacro:unless value="${joint_limited}">
-        <limit lower="${-2.0 * pi}" upper="${2.0 * pi}" effort="330.0" velocity="2.16"/>
-      </xacro:unless>
-      <xacro:if value="${joint_limited}">
-        <limit lower="${shoulder_pan_lower_limit}" upper="${shoulder_pan_upper_limit}" effort="330.0" velocity="2.16"/>
+        <limit lower="${-2.0 * pi}" upper="${2.0 * pi}" effort="330.0" velocity="2.0"/>
+      </xacro:unless>
+      <xacro:if value="${joint_limited}">
+        <limit lower="${shoulder_pan_lower_limit}" upper="${shoulder_pan_upper_limit}" effort="330.0" velocity="2.0"/>
       </xacro:if>
       <dynamics damping="0.0" friction="0.0"/>
@@ -115,8 +115,8 @@
       <axis xyz="0 1 0" />
       <xacro:unless value="${joint_limited}">
-        <limit lower="${-2.0 * pi}" upper="${2.0 * pi}" effort="330.0" velocity="2.16"/>
-      </xacro:unless>
-      <xacro:if value="${joint_limited}">
-        <limit lower="${shoulder_lift_lower_limit}" upper="${shoulder_lift_upper_limit}" effort="330.0" velocity="2.16"/>
+        <limit lower="${-2.0 * pi}" upper="${2.0 * pi}" effort="330.0" velocity="2.0"/>
+      </xacro:unless>
+      <xacro:if value="${joint_limited}">
+        <limit lower="${shoulder_lift_lower_limit}" upper="${shoulder_lift_upper_limit}" effort="330.0" velocity="2.0"/>
       </xacro:if>
       <dynamics damping="0.0" friction="0.0"/>
@@ -146,8 +146,8 @@
       <axis xyz="0 1 0" />
       <xacro:unless value="${joint_limited}">
-        <limit lower="${-pi}" upper="${pi}" effort="150.0" velocity="3.15"/>
-      </xacro:unless>
-      <xacro:if value="${joint_limited}">
-        <limit lower="${elbow_joint_lower_limit}" upper="${elbow_joint_upper_limit}" effort="150.0" velocity="3.15"/>
+        <limit lower="${-2.0 * pi}" upper="${2.0 * pi}" effort="150.0" velocity="2.0"/>
+      </xacro:unless>
+      <xacro:if value="${joint_limited}">
+        <limit lower="${elbow_joint_lower_limit}" upper="${elbow_joint_upper_limit}" effort="150.0" velocity="2.0"/>
       </xacro:if>
       <dynamics damping="0.0" friction="0.0"/>
@@ -177,8 +177,8 @@
       <axis xyz="0 1 0" />
       <xacro:unless value="${joint_limited}">
-        <limit lower="${-2.0 * pi}" upper="${2.0 * pi}" effort="54.0" velocity="3.2"/>
-      </xacro:unless>
-      <xacro:if value="${joint_limited}">
-        <limit lower="${wrist_1_lower_limit}" upper="${wrist_1_upper_limit}" effort="54.0" velocity="3.2"/>
+        <limit lower="${-2.0 * pi}" upper="${2.0 * pi}" effort="54.0" velocity="2.0"/>
+      </xacro:unless>
+      <xacro:if value="${joint_limited}">
+        <limit lower="${wrist_1_lower_limit}" upper="${wrist_1_upper_limit}" effort="54.0" velocity="2.0"/>
       </xacro:if>
       <dynamics damping="0.0" friction="0.0"/>
@@ -208,8 +208,8 @@
       <axis xyz="0 0 1" />
       <xacro:unless value="${joint_limited}">
-        <limit lower="${-2.0 * pi}" upper="${2.0 * pi}" effort="54.0" velocity="3.2"/>
-      </xacro:unless>
-      <xacro:if value="${joint_limited}">
-        <limit lower="${wrist_2_lower_limit}" upper="${wrist_2_upper_limit}" effort="54.0" velocity="3.2"/>
+        <limit lower="${-2.0 * pi}" upper="${2.0 * pi}" effort="54.0" velocity="2.0"/>
+      </xacro:unless>
+      <xacro:if value="${joint_limited}">
+        <limit lower="${wrist_2_lower_limit}" upper="${wrist_2_upper_limit}" effort="54.0" velocity="2.0"/>
       </xacro:if>
       <dynamics damping="0.0" friction="0.0"/>
@@ -239,8 +239,8 @@
       <axis xyz="0 1 0" />
       <xacro:unless value="${joint_limited}">
-        <limit lower="${-2.0 * pi}" upper="${2.0 * pi}" effort="54.0" velocity="3.2"/>
-      </xacro:unless>
-      <xacro:if value="${joint_limited}">
-        <limit lower="${wrist_3_lower_limit}" upper="${wrist_3_upper_limit}" effort="54.0" velocity="3.2"/>
+        <limit lower="${-2.0 * pi}" upper="${2.0 * pi}" effort="54.0" velocity="2.0"/>
+      </xacro:unless>
+      <xacro:if value="${joint_limited}">
+        <limit lower="${wrist_3_lower_limit}" upper="${wrist_3_upper_limit}" effort="54.0" velocity="2.0"/>
       </xacro:if>
       <dynamics damping="0.0" friction="0.0"/>

Commit message: change urdf joint limits

File: ur_description/urdf/ur10.urdf.xacro (robot description, xacro)
@@ -53,6 +53,15 @@
     </inertial>
   </xacro:macro>
+  <!-- before changing arm position, before 19.02.2020
   <xacro:macro name="ur10_robot" params="prefix joint_limited
 		 shoulder_pan_lower_limit:=${-0.5*pi}    shoulder_pan_upper_limit:=${2.75}
+		 shoulder_lift_lower_limit:=${-pi}    shoulder_lift_upper_limit:=${pi}
+		 elbow_joint_lower_limit:=${-pi}    elbow_joint_upper_limit:=${0.2}
+		 wrist_1_lower_limit:=${-2*pi}    wrist_1_upper_limit:=${-0.5}
+		 wrist_2_lower_limit:=${-pi}    wrist_2_upper_limit:=${pi}
+		 wrist_3_lower_limit:=${0.5-pi}    wrist_3_upper_limit:=${0.5*pi}">
+  -->
+  <xacro:macro name="ur10_robot" params="prefix joint_limited
+		 shoulder_pan_lower_limit:=${-4.80}    shoulder_pan_upper_limit:=${0.0}
 		 shoulder_lift_lower_limit:=${-pi}    shoulder_lift_upper_limit:=${pi}
 		 elbow_joint_lower_limit:=${-pi}    elbow_joint_upper_limit:=${0.2}

Commit message: change link names

File: ur_description/urdf/ur10.urdf.xacro (robot description, xacro)
@@ -80,5 +80,5 @@
     <joint name="${prefix}1_joint" type="revolute">
       <parent link="${prefix}base_link" />
-      <child link = "${prefix}shoulder_link" />
+      <child link = "${prefix}1_link" />
       <origin xyz="0.0 0.0 ${shoulder_height}" rpy="0.0 0.0 0.0" />
       <axis xyz="0 0 1" />
@@ -91,5 +91,5 @@
       <dynamics damping="0.0" friction="0.0"/>
     </joint>
-    <link name="${prefix}shoulder_link">
+    <link name="${prefix}1_link">
       <visual>
         <geometry>
@@ -110,6 +110,6 @@
     </link>
     <joint name="${prefix}2_joint" type="revolute">
-      <parent link="${prefix}shoulder_link" />
-      <child link = "${prefix}upper_arm_link" />
+      <parent link="${prefix}1_link" />
+      <child link = "${prefix}2_link" />
       <origin xyz="0.0 ${shoulder_offset} 0.0" rpy="0.0 ${pi / 2.0} 0.0" />
       <axis xyz="0 1 0" />
@@ -122,5 +122,5 @@
       <dynamics damping="0.0" friction="0.0"/>
     </joint>
-    <link name="${prefix}upper_arm_link">
+    <link name="${prefix}2_link">
       <visual>
         <geometry>
@@ -141,6 +141,6 @@
     </link>
     <joint name="${prefix}3_joint" type="revolute">
-      <parent link="${prefix}upper_arm_link" />
-      <child link = "${prefix}forearm_link" />
+      <parent link="${prefix}2_link" />
+      <child link = "${prefix}3_link" />
       <origin xyz="0.0 ${elbow_offset} ${upper_arm_length}" rpy="0.0 0.0 0.0" />
       <axis xyz="0 1 0" />
@@ -153,5 +153,5 @@
       <dynamics damping="0.0" friction="0.0"/>
     </joint>
-    <link name="${prefix}forearm_link">
+    <link name="${prefix}3_link">
       <visual>
          <geometry>
@@ -172,6 +172,6 @@
     </link>
     <joint name="${prefix}4_joint" type="revolute">
-      <parent link="${prefix}forearm_link" />
-      <child link = "${prefix}wrist_1_link" />
+      <parent link="${prefix}3_link" />
+      <child link = "${prefix}4_link" />
       <origin xyz="0.0 0.0 ${forearm_length}" rpy="0.0 ${pi / 2.0} 0.0" />
       <axis xyz="0 1 0" />
@@ -184,5 +184,5 @@
       <dynamics damping="0.0" friction="0.0"/>
     </joint>
-    <link name="${prefix}wrist_1_link">
+    <link name="${prefix}4_link">
       <visual>
         <geometry>
@@ -203,6 +203,6 @@
     </link>
     <joint name="${prefix}5_joint" type="revolute">
-      <parent link="${prefix}wrist_1_link" />
-      <child link = "${prefix}wrist_2_link" />
+      <parent link="${prefix}4_link" />
+      <child link = "${prefix}5_link" />
       <origin xyz="0.0 ${wrist_1_length} 0.0" rpy="0.0 0.0 0.0" />
       <axis xyz="0 0 1" />
@@ -215,5 +215,5 @@
       <dynamics damping="0.0" friction="0.0"/>
     </joint>
-    <link name="${prefix}wrist_2_link">
+    <link name="${prefix}5_link">
       <visual>
         <geometry>
@@ -234,6 +234,6 @@
     </link>
     <joint name="${prefix}6_joint" type="revolute">
-      <parent link="${prefix}wrist_2_link" />
-      <child link = "${prefix}wrist_3_link" />
+      <parent link="${prefix}5_link" />
+      <child link = "${prefix}6_link" />
       <origin xyz="0.0 0.0 ${wrist_2_length}" rpy="0.0 0.0 0.0" />
       <axis xyz="0 1 0" />
@@ -246,5 +246,5 @@
       <dynamics damping="0.0" friction="0.0"/>
     </joint>
-    <link name="${prefix}wrist_3_link">
+    <link name="${prefix}6_link">
       <visual>
         <geometry>
@@ -265,5 +265,5 @@
     </link>
     <joint name="${prefix}ee_fixed_joint" type="fixed">
-      <parent link="${prefix}wrist_3_link" />
+      <parent link="${prefix}6_link" />
       <child link = "${prefix}ee_link" />
       <origin xyz="0.0 ${wrist_3_length} 0.0" rpy="0.0 0.0 ${pi/2.0}" />
@@ -301,5 +301,5 @@
     <joint name="${prefix}wrist_3_link-tool0_fixed_joint" type="fixed">
       <origin xyz="0.0 ${wrist_3_length+0.14} 0.0" rpy="0.0 0.0 ${pi/2.0}" />
-      <parent link="${prefix}wrist_3_link"/>
+      <parent link="${prefix}6_link"/>
       <child link="${prefix}tool0"/>
       <xacro:unless value="${joint_limited}">

Commit message: change jointname and config

File: ur_description/urdf/ur10.urdf.xacro (robot description, xacro)
@@ -78,5 +78,5 @@
       </xacro:cylinder_inertial>
     </link>
-    <joint name="${prefix}shoulder_pan_joint" type="revolute">
+    <joint name="${prefix}1_joint" type="revolute">
       <parent link="${prefix}base_link" />
       <child link = "${prefix}shoulder_pan_link" />
@@ -109,5 +109,5 @@
       </xacro:cylinder_inertial>
     </link>
-    <joint name="${prefix}shoulder_lift_joint" type="revolute">
+    <joint name="${prefix}2_joint" type="revolute">
       <parent link="${prefix}shoulder_pan_link" />
       <child link = "${prefix}shoulder_lift_link" />
@@ -140,5 +140,5 @@
       </xacro:cylinder_inertial>
     </link>
-    <joint name="${prefix}elbow_joint" type="revolute">
+    <joint name="${prefix}3_joint" type="revolute">
       <parent link="${prefix}shoulder_lift_link" />
       <child link = "${prefix}elbow_link" />
@@ -171,5 +171,5 @@
       </xacro:cylinder_inertial>
     </link>
-    <joint name="${prefix}wrist_1_joint" type="revolute">
+    <joint name="${prefix}4_joint" type="revolute">
       <parent link="${prefix}elbow_link" />
       <child link = "${prefix}wrist_1_link" />
@@ -202,5 +202,5 @@
       </xacro:cylinder_inertial>
     </link>
-    <joint name="${prefix}wrist_2_joint" type="revolute">
+    <joint name="${prefix}5_joint" type="revolute">
       <parent link="${prefix}wrist_1_link" />
       <child link = "${prefix}wrist_2_link" />
@@ -233,5 +233,5 @@
       </xacro:cylinder_inertial>
     </link>
-    <joint name="${prefix}wrist_3_joint" type="revolute">
+    <joint name="${prefix}6_joint" type="revolute">
       <parent link="${prefix}wrist_2_link" />
       <child link = "${prefix}wrist_3_link" />

File: ur_description/urdf/ur10_joint_limited_robot.urdf.xacro (robot description, xacro)
@@ -6,4 +6,5 @@
   <!-- ur10 -->
   <xacro:include filename="$(find ur_description)/urdf/ur10.urdf.xacro" />
+    <!--
     <link name="world" />
     <joint name="world_joint" type="fixed">
@@ -12,6 +13,7 @@
       <origin xyz="0.0 0.0 0.0" rpy="0.0 0.0 0.0" />
     </joint>
+    -->
     <!-- inlcuding table top robot arm -->
-    <!--link name="world" />
+    <link name="world" />
     <joint name="world-robot_base_joint" type="fixed">
       <origin xyz="-0.65 -0.45 0.45" rpy="0 0 0" />
@@ -34,5 +36,5 @@
       <child link = "arm_base_link" />
       <origin xyz="0.0 0.0 0.45" rpy="0.0 0.0 -2.3562" />
-    </joint-->
+    </joint>
   <!-- arm -->
   <xacro:ur10_robot prefix="arm_" joint_limited="true"

File: ur_description/urdf/ur10_robot.urdf.xacro (robot description, xacro)
@@ -6,4 +6,5 @@
   <!-- ur10 -->
   <xacro:include filename="$(find ur_description)/urdf/ur10.urdf.xacro" />
+  <!--
   <link name="world" />
   <joint name="world_joint" type="fixed">
@@ -12,6 +13,7 @@
     <origin xyz="0.0 0.0 0.0" rpy="0.0 0.0 0.0" />
   </joint>
+  -->
  <!-- inlcuding table top robot arm -->
- <!--link name="world" />
+ <link name="world" />
   <joint name="world-robot_base_joint" type="fixed">
     <origin xyz="-0.65 -0.45 0.45" rpy="0 0 0" />
@@ -34,5 +36,5 @@
     <child link = "arm_base_link" />
     <origin xyz="0.0 0.0 0.45" rpy="0.0 0.0 -2.3562" />
-  </joint-->
+  </joint>
   <!-- arm -->
   <xacro:ur10_robot prefix="arm_" joint_limited="false"/>

Commit message: change joint limits based on order-picking robot

File: ur_description/urdf/ur10.urdf.xacro (robot description, xacro)
@@ -54,5 +54,5 @@
   </xacro:macro>
   <xacro:macro name="ur10_robot" params="prefix joint_limited
-		 shoulder_pan_lower_limit:=${-0.5*pi}    shoulder_pan_upper_limit:=${0.2}
+		 shoulder_pan_lower_limit:=${-0.5*pi}    shoulder_pan_upper_limit:=${2.75}
 		 shoulder_lift_lower_limit:=${-pi}    shoulder_lift_upper_limit:=${pi}
 		 elbow_joint_lower_limit:=${-pi}    elbow_joint_upper_limit:=${0.2}

File: ur_description/urdf/ur10_joint_limited_robot.urdf.xacro (robot description, xacro)
@@ -6,43 +6,18 @@
   <!-- ur10 -->
   <xacro:include filename="$(find ur_description)/urdf/ur10.urdf.xacro" />
-    <!--
-    <link name="world" />
-    <joint name="world_joint" type="fixed">
-      <parent link="world" />
-      <child link = "arm_base_link" />
-      <origin xyz="0.0 0.0 0.0" rpy="0.0 0.0 0.0" />
-    </joint>
-    -->
-    <!-- inlcuding table top robot arm -->
-    <link name="world" />
-    <joint name="world-robot_base_joint" type="fixed">
-      <origin xyz="-0.65 -0.45 0.45" rpy="0 0 0" />
-      <parent link="world"/>
-      <child link="robot_base"/>
-    </joint>
-    <link name="robot_base">
-        <visual>
-          <origin rpy="0 0 0" xyz="0 0 0"/>
-          <geometry>
-            <box size="1.30 0.90 0.90"/>
-          </geometry>
-          <material name="LightGrey">
-            <color rgba="0.7 0.7 0.7 1.0"/>
-          </material>
-        </visual>
-    </link>
-    <joint name="world_joint" type="fixed">
-      <parent link="robot_base" />
-      <child link = "base_link" />
-      <origin xyz="0.0 0.0 0.45" rpy="0.0 0.0 -2.3562" />
-    </joint>
+  <link name="world" />
+  <joint name="world_joint" type="fixed">
+    <parent link="world" />
+    <child link = "base_link" />
+    <origin xyz="0.0 0.0 0.0" rpy="0.0 0.0 0.0" />
+  </joint>
   <!-- arm -->
   <xacro:ur10_robot prefix="" joint_limited="true"
-               shoulder_pan_lower_limit="${-pi}" shoulder_pan_upper_limit="${pi}"
+               shoulder_pan_lower_limit="${-pi}" shoulder_pan_upper_limit="${2.75}"
                shoulder_lift_lower_limit="${-pi}" shoulder_lift_upper_limit="${pi}"
-               elbow_joint_lower_limit="${-pi}" elbow_joint_upper_limit="${pi}"
-               wrist_1_lower_limit="${-pi}" wrist_1_upper_limit="${pi}"
+               elbow_joint_lower_limit="${-pi}" elbow_joint_upper_limit="${0.2}"
+               wrist_1_lower_limit="${-2*pi}" wrist_1_upper_limit="${-0.5}"
                wrist_2_lower_limit="${-pi}" wrist_2_upper_limit="${pi}"
-               wrist_3_lower_limit="${-pi}" wrist_3_upper_limit="${pi}"
+               wrist_3_lower_limit="${0.5-pi}" wrist_3_upper_limit="${0.5*pi}"
   />
   <!-- ros_control plugin -->

Commit message: remove robotiq gripper and add just frame of gripper

File: ur_description/urdf/ur10.urdf.xacro (robot description, xacro)
@@ -311,4 +311,17 @@
       <dynamics damping="0.0" friction="0.0"/>
     </joint>
+    <joint name="${prefix}gripper_fixed_joint" type="fixed">
+      <parent link="${prefix}ee_link" />
+      <child link = "gripper" />
+      <origin xyz=" 0.1500 0.0 0.0" rpy="3.1415 0 0"/>
+    </joint>
+    <link name="gripper">
+      <collision>
+        <geometry>
+          <box size="0.01 0.01 0.01"/>
+        </geometry>
+        <origin rpy="0 0 0" xyz="-0.01 0 0"/>
+      </collision>
+    </link>
   </xacro:macro>
 </robot>
