Commit message: schmalz gripper added on robot

File: ur_e_description/urdf/ur5e_robot.urdf.xacro (robot description, xacro)
@@ -6,6 +6,6 @@
   <!-- ur5e -->
   <xacro:include filename="$(find ur_e_description)/urdf/ur5e.urdf.xacro" />
-  <!-- arm -->
-  <xacro:ur5e_robot prefix="" joint_limited="false"/>
+  <!-- Schmalz gripper -->
+  <xacro:include filename="$(find ur_e_description)/urdf/gripper.urdf.xacro" />
   <link name="world" />
   <joint name="world_joint" type="fixed">
@@ -14,3 +14,9 @@
     <origin xyz="0.0 0.0 0.0" rpy="0.0 0.0 0.0" />
   </joint>
+  <!-- arm -->
+  <xacro:ur5e_robot prefix="" joint_limited="false"/>
+  <!-- gripper -->
+  <xacro:vacuum_gripper name="gripper" parent="ee_link">
+    <origin xyz="0.074 0.0 0.0" rpy="0.0 0.0 1.57079632679" />
+  </xacro:vacuum_gripper>
 </robot>

Commit message: correct gripper orientation as x pointing to object

File: ur_e_description/urdf/ur5e_robot.urdf.xacro (robot description, xacro)
@@ -21,5 +21,5 @@
     <parent link="tool0" />
     <child link = "gripper" />
-    <origin xyz="0.0 0.0 0.105" rpy="0.0 0.0 0.0" />
+    <origin xyz="0.0 0.0 0.105" rpy="3.14 -1.57 0.0" />
   </joint>
 </robot>
